Commit message: feat(simulation): add IMU and camera sensor support
- Add IMU link/joint to URDF (Yahboom MPU9250); parse serial packets
  0x61/0x62/0x63 in yahboom_controller_node and publish /imu/data
- Add Gazebo camera sensor on camera_link (640x480, 30fps, 60° FOV)
  publishing /camera/image_raw; bridge both image and camera_info to ROS
- Create omnibot_world.sdf with gz-sim-sensors-system and gz-sim-imu-system
  as world-level plugins (required for camera rendering in Gazebo Harmonic)
- Update simulation.launch.py to use omnibot_world.sdf instead of empty.sdf
- Add Camera Image display and IMU Axes display to omnibot.rviz

Co-Authored-By: Claude Sonnet 4.6 <noreply@anthropic.com>

File: robot_ws/src/omnibot_description/urdf/omnibot.urdf.xacro (robot description, xacro)
@@ -70,4 +70,48 @@
         <child link="camera_link"/>
         <origin xyz="${camera_x_offset} ${camera_y_offset} ${camera_z_offset}" rpy="0 0 0"/> </joint>
+    <!-- Gazebo Camera Sensor — mounted on camera_link, publishes /camera/image_raw -->
+    <gazebo reference="camera_link">
+        <sensor name="camera_sensor" type="camera">
+            <always_on>1</always_on>
+            <update_rate>30</update_rate>
+            <visualize>false</visualize>
+            <topic>/camera/image_raw</topic>
+            <gz_frame_id>camera_link</gz_frame_id>
+            <camera>
+                <horizontal_fov>1.047</horizontal_fov> <!-- 60 deg -->
+                <image>
+                    <width>640</width>
+                    <height>480</height>
+                    <format>R8G8B8</format>
+                </image>
+                <clip>
+                    <near>0.05</near>
+                    <far>50</far>
+                </clip>
+            </camera>
+        </sensor>
+    </gazebo>
+    <!-- IMU Link — represents the Yahboom board's built-in MPU9250 (9-axis IMU) -->
+    <link name="imu_link">
+        <visual>
+            <origin xyz="0 0 0" rpy="0 0 0"/>
+            <geometry><box size="0.03 0.03 0.015"/></geometry>
+            <material name="red"><color rgba="0.8 0.1 0.1 1"/></material>
+        </visual>
+        <collision>
+            <origin xyz="0 0 0" rpy="0 0 0"/>
+            <geometry><box size="0.03 0.03 0.015"/></geometry>
+        </collision>
+        <inertial>
+            <mass value="0.01"/>
+            <origin xyz="0 0 0" rpy="0 0 0"/>
+            <inertia ixx="1e-6" ixy="0" ixz="0" iyy="1e-6" iyz="0" izz="1e-6"/>
+        </inertial>
+    </link>
+    <joint name="imu_joint" type="fixed">
+        <parent link="base_link"/>
+        <child link="imu_link"/>
+        <origin xyz="0 0 0" rpy="0 0 0"/>
+    </joint>
     <xacro:macro name="wheel" params="prefix x_reflect y_reflect yaw_reflect">
         <link name="${prefix}_wheel_link">
@@ -117,4 +161,26 @@
     </xacro:macro>
     <xacro:wheel prefix="front_left"  x_reflect="1"  y_reflect="1"  yaw_reflect="1"/>   <xacro:wheel prefix="front_right" x_reflect="1"  y_reflect="-1" yaw_reflect="-1"/>  <xacro:wheel prefix="rear_left"   x_reflect="-1" y_reflect="1"  yaw_reflect="-1"/>  <xacro:wheel prefix="rear_right"  x_reflect="-1" y_reflect="-1" yaw_reflect="1"/>
+    <!-- Gazebo IMU Sensor — publishes /imu/data as gz.msgs.IMU -->
+    <gazebo reference="imu_link">
+        <sensor name="imu_sensor" type="imu">
+            <always_on>1</always_on>
+            <update_rate>100</update_rate>
+            <visualize>false</visualize>
+            <topic>/imu/data</topic>
+            <gz_frame_id>imu_link</gz_frame_id>
+            <imu>
+                <angular_velocity>
+                    <x><noise type="gaussian"><mean>0</mean><stddev>0.002</stddev></noise></x>
+                    <y><noise type="gaussian"><mean>0</mean><stddev>0.002</stddev></noise></y>
+                    <z><noise type="gaussian"><mean>0</mean><stddev>0.002</stddev></noise></z>
+                </angular_velocity>
+                <linear_acceleration>
+                    <x><noise type="gaussian"><mean>0</mean><stddev>0.017</stddev></noise></x>
+                    <y><noise type="gaussian"><mean>0</mean><stddev>0.017</stddev></noise></y>
+                    <z><noise type="gaussian"><mean>0</mean><stddev>0.017</stddev></noise></z>
+                </linear_acceleration>
+            </imu>
+        </sensor>
+    </gazebo>
     <!-- Gazebo Harmonic Mecanum Drive Plugin -->
     <gazebo>
@@ -143,4 +209,6 @@
             <joint_name>rear_right_wheel_joint</joint_name>
         </plugin>
+        <!-- NOTE: gz-sim-sensors-system and gz-sim-imu-system are world-level
+             plugins loaded in omnibot_world.sdf — do NOT duplicate here. -->
     </gazebo>
 </robot>
