Commit message: feat: redesign URDF to match real robot — two-plate chassis + SO-ARM 101
Chassis:
- Replace single-box chassis with two 6mm aluminium plates separated by
  8 hex standoffs (160mm apart), matching the real robot structure
- Ground clearance corrected from 30mm → 70mm (total height ~242mm)
- Both plates black (0.08 0.08 0.08), replacing previous blue

Cameras:
- Move 4× OV9732 cameras from top-edge to side-face of top plate
  (flush-mounted in camera cases, facing outward)
- Relocate Orbbec Astra Pro depth camera from front to rear of top plate,
  facing rearward — robot drives backward during Nav2 navigation so the
  depth camera covers the direction of travel

SO-ARM 101:
- Add full 6-DOF SO-ARM 101 kinematic chain with correct joint origins
  and limits sourced from the official TheRobotStudio so101_new_calib.urdf
- Joints: shoulder_pan, shoulder_lift, elbow_flex, wrist_flex, wrist_roll,
  gripper — all with proper revolute limits and transmissions
- Visuals: simplified box/cylinder primitives (no STL meshes required)
  with white for 3D-printed PLA parts, dark for STS3215 servos
- Mounted at front-centre of top plate

Viewer:
- Rewrite urdf_viewer.html to reflect new two-plate design, standoffs,
  arm, rear depth camera, and side-mounted OV9732 cameras
- Add arm pose cycling and arm visibility toggle buttons

Co-Authored-By: Claude Sonnet 4.6 <noreply@anthropic.com>

File: robot_ws/src/omnibot_description/urdf/omnibot.urdf.xacro (robot description, xacro)
@@ -2,20 +2,63 @@
 <robot xmlns:xacro="http://www.ros.org/wiki/xacro" name="mecanum_bot">
     <xacro:property name="PI" value="3.1415926535897931"/>
-    <xacro:property name="chassis_length" value="0.265"/>
-    <xacro:property name="chassis_width" value="0.25"/>
-    <xacro:property name="chassis_height" value="0.18"/> <xacro:property name="ground_clearance" value="0.03"/>
-    <xacro:property name="wheel_radius" value="0.04"/>
-    <xacro:property name="wheel_width" value="0.037"/>
-    <xacro:property name="wheel_separation_x" value="0.165"/> <xacro:property name="wheel_separation_y" value="0.215"/> <xacro:property name="base_link_z_offset" value="${ground_clearance + chassis_height / 2.0}"/> <xacro:property name="wheel_z_offset" value="${wheel_radius - base_link_z_offset}"/> <xacro:property name="wheel_x_offset" value="${wheel_separation_x / 2.0}"/>
-    <xacro:property name="wheel_y_offset" value="${wheel_separation_y / 2.0}"/>
-    <xacro:property name="camera_x_offset" value="0"/> <xacro:property name="camera_y_offset" value="0"/> <xacro:property name="camera_z_offset" value="${chassis_height / 2.0 + 0.01}"/> <xacro:property name="camera_size_x" value="0.04"/> <xacro:property name="camera_size_y" value="0.025"/> <xacro:property name="camera_size_z" value="0.025"/> <xacro:property name="base_mass" value="2.5"/> <xacro:property name="wheel_mass" value="0.2"/> <xacro:property name="camera_mass" value="0.05"/> <link name="base_footprint"/>
+    <!-- ================================================================
+         Chassis — two black aluminium plates separated by 8 standoffs.
+         Bottom plate = base_link.
+         Total height (ground → top plate surface) ≈ 240 mm.
+         ================================================================ -->
+    <xacro:property name="chassis_length"    value="0.265"/>  <!-- 265 mm front-to-rear -->
+    <xacro:property name="chassis_width"     value="0.250"/>  <!-- 250 mm left-to-right -->
+    <xacro:property name="plate_thickness"   value="0.006"/>  <!-- 6 mm aluminium plate -->
+    <xacro:property name="standoff_height"   value="0.160"/>  <!-- 160 mm between plate faces -->
+    <xacro:property name="ground_clearance"  value="0.070"/>  <!-- ground → bottom of bottom plate -->
+    <!-- Bottom plate (base_link) centre above base_footprint -->
+    <xacro:property name="base_link_z_offset" value="${ground_clearance + plate_thickness / 2.0}"/>
+    <!-- Top plate centre above base_link centre -->
+    <xacro:property name="top_plate_dz"       value="${plate_thickness + standoff_height}"/>
+    <!-- Top surface of top plate above base_link centre (used for mounting) -->
+    <xacro:property name="top_surface_dz"     value="${top_plate_dz + plate_thickness / 2.0}"/>
+    <!-- ================================================================
+         Wheels
+         ================================================================ -->
+    <xacro:property name="wheel_radius"       value="0.04"/>
+    <xacro:property name="wheel_width"        value="0.037"/>
+    <xacro:property name="wheel_separation_x" value="0.165"/>
+    <xacro:property name="wheel_separation_y" value="0.215"/>
+    <!-- Negative: wheels hang below bottom plate -->
+    <xacro:property name="wheel_z_offset"     value="${wheel_radius - base_link_z_offset}"/>
+    <xacro:property name="wheel_x_offset"     value="${wheel_separation_x / 2.0}"/>
+    <xacro:property name="wheel_y_offset"     value="${wheel_separation_y / 2.0}"/>
+    <!-- ================================================================
+         Masses
+         ================================================================ -->
+    <xacro:property name="base_mass"       value="1.5"/>
+    <xacro:property name="top_plate_mass"  value="1.0"/>
+    <xacro:property name="wheel_mass"      value="0.2"/>
+    <xacro:property name="camera_mass"     value="0.05"/>
+    <xacro:property name="astra_mass"      value="0.300"/>
+    <!-- ================================================================
+         OV9732 camera body size (camera + case)
+         ================================================================ -->
+    <xacro:property name="camera_size_x"   value="0.030"/>  <!-- depth into face -->
+    <xacro:property name="camera_size_y"   value="0.030"/>  <!-- width -->
+    <xacro:property name="camera_size_z"   value="0.025"/>  <!-- height -->
+    <!-- ================================================================
+         base_footprint — ground-level reference frame
+         ================================================================ -->
+    <link name="base_footprint"/>
+    <!-- ================================================================
+         base_link — BOTTOM PLATE (black aluminium)
+         Thin flat plate at ground_clearance height above ground.
+         Electronics, Pi, battery, and Yahboom board are mounted
+         between the two plates (not modelled individually).
+         ================================================================ -->
     <link name="base_link">
         <visual>
             <origin xyz="0 0 0" rpy="0 0 0"/>
             <geometry>
-                <box size="${chassis_length} ${chassis_width} ${chassis_height}"/>
-            </geometry>
-            <material name="blue">
-                <color rgba="0.2 0.4 0.8 1"/>
+                <box size="${chassis_length} ${chassis_width} ${plate_thickness}"/>
+            </geometry>
+            <material name="chassis_black">
+                <color rgba="0.08 0.08 0.08 1"/>
             </material>
         </visual>
@@ -23,5 +66,5 @@
             <origin xyz="0 0 0" rpy="0 0 0"/>
             <geometry>
-                <box size="${chassis_length} ${chassis_width} ${chassis_height}"/>
+                <box size="${chassis_length} ${chassis_width} ${plate_thickness}"/>
             </geometry>
         </collision>
@@ -29,11 +72,14 @@
             <mass value="${base_mass}"/>
             <origin xyz="0 0 0" rpy="0 0 0"/>
-            <inertia ixx="${base_mass / 12.0 * (chassis_width*chassis_width + chassis_height*chassis_height)}" ixy="0.0" ixz="0.0"
-                     iyy="${base_mass / 12.0 * (chassis_length*chassis_length + chassis_height*chassis_height)}" iyz="0.0"
-                     izz="${base_mass / 12.0 * (chassis_length*chassis_length + chassis_width*chassis_width)}" />
+            <inertia
+                ixx="${base_mass / 12.0 * (chassis_width*chassis_width   + plate_thickness*plate_thickness)}"
+                ixy="0" ixz="0"
+                iyy="${base_mass / 12.0 * (chassis_length*chassis_length + plate_thickness*plate_thickness)}"
+                iyz="0"
+                izz="${base_mass / 12.0 * (chassis_length*chassis_length + chassis_width*chassis_width)}"/>
         </inertial>
     </link>
     <gazebo reference="base_link">
-        <material>Gazebo/Blue</material>
+        <material>Gazebo/DarkGrey</material>
     </gazebo>
     <joint name="base_footprint_joint" type="fixed">
@@ -43,8 +89,90 @@
     </joint>
     <!-- ================================================================
-         Base camera macro — instantiated 4× for front/rear/left/right.
-         OV9732: 100° FOV (1.745 rad), 1280×720, USB UVC.
-         Each camera sits on the top edge of the chassis, tilted ~30°
-         downward toward the ground plane for BEV capture.
+         Standoffs — 8 aluminium hex standoffs connecting the two plates.
+         Two pairs at each corner region of the chassis.
+         ================================================================ -->
+    <xacro:macro name="standoff" params="prefix x_pos y_pos">
+        <link name="${prefix}_standoff_link">
+            <visual>
+                <origin xyz="0 0 0" rpy="0 0 0"/>
+                <geometry>
+                    <cylinder radius="0.007" length="${standoff_height}"/>
+                </geometry>
+                <material name="standoff_silver">
+                    <color rgba="0.65 0.65 0.65 1"/>
+                </material>
+            </visual>
+            <collision>
+                <origin xyz="0 0 0" rpy="0 0 0"/>
+                <geometry>
+                    <cylinder radius="0.007" length="${standoff_height}"/>
+                </geometry>
+            </collision>
+            <inertial>
+                <mass value="0.04"/>
+                <origin xyz="0 0 0" rpy="0 0 0"/>
+                <inertia ixx="0.0001" ixy="0" ixz="0" iyy="0.0001" iyz="0" izz="0.0001"/>
+            </inertial>
+        </link>
+        <joint name="${prefix}_standoff_joint" type="fixed">
+            <parent link="base_link"/>
+            <child link="${prefix}_standoff_link"/>
+            <!-- standoff spans from top face of bottom plate to bottom face of top plate -->
+            <origin xyz="${x_pos} ${y_pos} ${plate_thickness / 2.0 + standoff_height / 2.0}" rpy="0 0 0"/>
+        </joint>
+    </xacro:macro>
+    <!-- 8 standoffs: two pairs near each corner -->
+    <xacro:standoff prefix="so_fl_a" x_pos=" 0.095" y_pos=" 0.085"/>
+    <xacro:standoff prefix="so_fl_b" x_pos=" 0.065" y_pos=" 0.095"/>
+    <xacro:standoff prefix="so_fr_a" x_pos=" 0.095" y_pos="-0.085"/>
+    <xacro:standoff prefix="so_fr_b" x_pos=" 0.065" y_pos="-0.095"/>
+    <xacro:standoff prefix="so_rl_a" x_pos="-0.095" y_pos=" 0.085"/>
+    <xacro:standoff prefix="so_rl_b" x_pos="-0.065" y_pos=" 0.095"/>
+    <xacro:standoff prefix="so_rr_a" x_pos="-0.095" y_pos="-0.085"/>
+    <xacro:standoff prefix="so_rr_b" x_pos="-0.065" y_pos="-0.095"/>
+    <!-- ================================================================
+         top_plate_link — UPPER PLATE (black aluminium)
+         The SO-ARM 101 and depth camera mount here.
+         ================================================================ -->
+    <link name="top_plate_link">
+        <visual>
+            <origin xyz="0 0 0" rpy="0 0 0"/>
+            <geometry>
+                <box size="${chassis_length} ${chassis_width} ${plate_thickness}"/>
+            </geometry>
+            <material name="chassis_black"/>
+        </visual>
+        <collision>
+            <origin xyz="0 0 0" rpy="0 0 0"/>
+            <geometry>
+                <box size="${chassis_length} ${chassis_width} ${plate_thickness}"/>
+            </geometry>
+        </collision>
+        <inertial>
+            <mass value="${top_plate_mass}"/>
+            <origin xyz="0 0 0" rpy="0 0 0"/>
+            <inertia
+                ixx="${top_plate_mass / 12.0 * (chassis_width*chassis_width   + plate_thickness*plate_thickness)}"
+                ixy="0" ixz="0"
+                iyy="${top_plate_mass / 12.0 * (chassis_length*chassis_length + plate_thickness*plate_thickness)}"
+                iyz="0"
+                izz="${top_plate_mass / 12.0 * (chassis_length*chassis_length + chassis_width*chassis_width)}"/>
+        </inertial>
+    </link>
+    <gazebo reference="top_plate_link">
+        <material>Gazebo/DarkGrey</material>
+    </gazebo>
+    <joint name="top_plate_joint" type="fixed">
+        <parent link="base_link"/>
+        <child link="top_plate_link"/>
+        <!-- top plate centre is one plate_thickness + standoff_height above bottom plate centre -->
+        <origin xyz="0 0 ${top_plate_dz}" rpy="0 0 0"/>
+    </joint>
+    <!-- ================================================================
+         OV9732 wide-angle cameras — one on each side face of the chassis.
+         Mounted flush with the side faces of the top plate inside a
+         camera case. Each camera faces outward with a 30° downward tilt
+         for ground-obstacle coverage.
+         FOV: 100° (1.745 rad), 1280×720, USB UVC.
          ================================================================ -->
     <xacro:macro name="base_camera" params="prefix x_pos y_pos yaw_angle">
@@ -56,5 +184,5 @@
                 </geometry>
                 <material name="dark_grey">
-                    <color rgba="0.2 0.2 0.2 1"/>
+                    <color rgba="0.15 0.15 0.15 1"/>
                 </material>
             </visual>
@@ -70,18 +198,17 @@
                 <inertia
                     ixx="${camera_mass / 12.0 * (camera_size_y*camera_size_y + camera_size_z*camera_size_z)}"
-                    ixy="0.0" ixz="0.0"
+                    ixy="0" ixz="0"
                     iyy="${camera_mass / 12.0 * (camera_size_x*camera_size_x + camera_size_z*camera_size_z)}"
-                    iyz="0.0"
+                    iyz="0"
                     izz="${camera_mass / 12.0 * (camera_size_x*camera_size_x + camera_size_y*camera_size_y)}"/>
             </inertial>
         </link>
-        <!-- Tilt 30° downward (pitch = -PI/6) so cameras look at the ground -->
+        <!-- Parent: top_plate_link. Cameras sit on the side faces, at plate level. -->
         <joint name="${prefix}_camera_joint" type="fixed">
-            <parent link="base_link"/>
+            <parent link="top_plate_link"/>
             <child link="${prefix}_camera_link"/>
-            <origin xyz="${x_pos} ${y_pos} ${chassis_height / 2.0 + 0.015}"
+            <origin xyz="${x_pos} ${y_pos} 0"
                     rpy="0 ${-PI/6} ${yaw_angle}"/>
         </joint>
-        <!-- Gazebo camera sensor for simulation — 100° FOV, 1280×720 -->
         <gazebo reference="${prefix}_camera_link">
             <sensor name="${prefix}_camera_sensor" type="camera">
@@ -92,5 +219,5 @@
                 <gz_frame_id>${prefix}_camera_link</gz_frame_id>
                 <camera>
-                    <horizontal_fov>1.745</horizontal_fov> <!-- 100 deg -->
+                    <horizontal_fov>1.745</horizontal_fov>
                     <image>
                         <width>640</width>
@@ -106,41 +233,38 @@
         </gazebo>
     </xacro:macro>
-    <!-- Instantiate 4 base cameras at the four edges of the chassis -->
-    <!-- Front: centre of forward edge, facing forward (yaw=0) -->
+    <!-- Cameras on the 4 side faces of the top plate -->
     <xacro:base_camera prefix="front"
-        x_pos="${chassis_length / 2.0 - 0.01}"
+        x_pos="${chassis_length / 2.0 + camera_size_x / 2.0}"
         y_pos="0"
         yaw_angle="0"/>
-    <!-- Rear: centre of rear edge, facing backward (yaw=PI) -->
     <xacro:base_camera prefix="rear"
-        x_pos="${-(chassis_length / 2.0 - 0.01)}"
+        x_pos="${-(chassis_length / 2.0 + camera_size_x / 2.0)}"
         y_pos="0"
         yaw_angle="${PI}"/>
-    <!-- Left: centre of left edge, facing left (yaw=PI/2) -->
     <xacro:base_camera prefix="left"
         x_pos="0"
-        y_pos="${chassis_width / 2.0 - 0.01}"
+        y_pos="${chassis_width / 2.0 + camera_size_x / 2.0}"
         yaw_angle="${PI/2}"/>
-    <!-- Right: centre of right edge, facing right (yaw=-PI/2) -->
     <xacro:base_camera prefix="right"
         x_pos="0"
-        y_pos="${-(chassis_width / 2.0 - 0.01)}"
+        y_pos="${-(chassis_width / 2.0 + camera_size_x / 2.0)}"
         yaw_angle="${-PI/2}"/>
     <!-- ================================================================
-         Wrist camera link — mounted on the arm end-effector.
-         Defined as a separate fixed link relative to wrist_link.
-         The arm URDF (omnibot_arm package) provides wrist_link; this
-         joint connects to it when the arm is loaded in the same URDF.
-         For standalone robot description without arm, this link is
-         kept as a child of base_link as a placeholder.
-         ================================================================ -->
-    <link name="wrist_camera_link">
-        <visual>
-            <origin xyz="0 0 0" rpy="0 0 0"/>
-            <geometry>
-                <box size="${camera_size_x} ${camera_size_y} ${camera_size_z}"/>
-            </geometry>
-            <material name="dark_grey_wrist">
-                <color rgba="0.2 0.2 0.2 1"/>
+         Orbbec Astra Pro Depth Camera
+         Mounted on the TOP PLATE, facing REARWARD (−X direction).
+         The robot drives backward for Nav2, so the depth camera covers
+         the direction of travel. Tilted 12° downward.
+         Astra Pro: 165 mm × 30 mm × 40 mm, 300 g, USB 2.0
+         Depth range: 0.6–8.0 m, FOV 60°H × 49.5°V
+         ================================================================ -->
+    <link name="depth_camera_link">
+        <visual>
+            <origin xyz="0 0 0" rpy="0 0 0"/>
+            <geometry>
+                <!-- 165 mm wide, 30 mm deep, 40 mm tall -->
+                <box size="0.030 0.165 0.040"/>
+            </geometry>
+            <material name="astra_black">
+                <color rgba="0.08 0.08 0.08 1"/>
             </material>
         </visual>
@@ -148,32 +272,67 @@
             <origin xyz="0 0 0" rpy="0 0 0"/>
             <geometry>
-                <box size="${camera_size_x} ${camera_size_y} ${camera_size_z}"/>
-            </geometry>
-        </collision>
-        <inertial>
-            <mass value="${camera_mass}"/>
+                <box size="0.030 0.165 0.040"/>
+            </geometry>
+        </collision>
+        <inertial>
+            <mass value="${astra_mass}"/>
             <origin xyz="0 0 0" rpy="0 0 0"/>
             <inertia
-                ixx="${camera_mass / 12.0 * (camera_size_y*camera_size_y + camera_size_z*camera_size_z)}"
-                ixy="0.0" ixz="0.0"
-                iyy="${camera_mass / 12.0 * (camera_size_x*camera_size_x + camera_size_z*camera_size_z)}"
-                iyz="0.0"
-                izz="${camera_mass / 12.0 * (camera_size_x*camera_size_x + camera_size_y*camera_size_y)}"/>
-        </inertial>
-    </link>
-    <!-- Placeholder joint: wrist camera on base_link until arm URDF is merged -->
-    <joint name="wrist_camera_joint" type="fixed">
-        <parent link="base_link"/>
-        <child link="wrist_camera_link"/>
-        <origin xyz="${chassis_length / 2.0 + 0.02} 0 ${chassis_height / 2.0 + 0.08}"
-                rpy="0 ${PI/4} 0"/>
-    </joint>
-    <!-- Gazebo simulation sensor — mounted on camera_link, publishes /camera/image_raw -->
-    <!-- Kept for backwards-compatibility with simulation.launch.py -->
+                ixx="${astra_mass / 12.0 * (0.165*0.165 + 0.040*0.040)}"
+                ixy="0" ixz="0"
+                iyy="${astra_mass / 12.0 * (0.030*0.030 + 0.040*0.040)}"
+                iyz="0"
+                izz="${astra_mass / 12.0 * (0.030*0.030 + 0.165*0.165)}"/>
+        </inertial>
+    </link>
+    <!-- Rear-centre of top plate, 20 mm above surface, 12° down-tilt, facing rearward (yaw=PI) -->
+    <joint name="depth_camera_joint" type="fixed">
+        <parent link="top_plate_link"/>
+        <child link="depth_camera_link"/>
+        <origin xyz="${-(chassis_length / 2.0 - 0.030)} 0 ${plate_thickness / 2.0 + 0.025}"
+                rpy="0 -0.2094 ${PI}"/>
+    </joint>
+    <!-- Optical frame: Z forward, X right, Y down (ROS convention) -->
+    <link name="depth_camera_optical_frame"/>
+    <joint name="depth_camera_optical_joint" type="fixed">
+        <parent link="depth_camera_link"/>
+        <child link="depth_camera_optical_frame"/>
+        <origin xyz="0 0 0" rpy="${-PI/2} 0 ${-PI/2}"/>
+    </joint>
+    <gazebo reference="depth_camera_link">
+        <sensor name="astra_pro_sensor" type="rgbd_camera">
+            <always_on>1</always_on>
+            <update_rate>30</update_rate>
+            <visualize>false</visualize>
+            <topic>/camera/depth</topic>
+            <gz_frame_id>depth_camera_optical_frame</gz_frame_id>
+            <camera>
+                <horizontal_fov>1.0472</horizontal_fov>
+                <image>
+                    <width>640</width>
+                    <height>480</height>
+                    <format>R_FLOAT32</format>
+                </image>
+                <clip>
+                    <near>0.6</near>
+                    <far>8.0</far>
+                </clip>
+                <noise>
+                    <type>gaussian</type>
+                    <mean>0.0</mean>
+                    <stddev>0.005</stddev>
+                </noise>
+            </camera>
+        </sensor>
+    </gazebo>
+    <!-- ================================================================
+         Backwards-compat camera_link for simulation.launch.py
+         Moved to top_plate centre, facing forward.
+         ================================================================ -->
     <link name="camera_link">
         <visual>
             <origin xyz="0 0 0" rpy="0 0 0"/>
             <geometry>
-                <box size="${camera_size_x} ${camera_size_y} ${camera_size_z}"/>
+                <box size="0.040 0.025 0.025"/>
             </geometry>
             <material name="grey">
@@ -183,25 +342,17 @@
         <collision>
             <origin xyz="0 0 0" rpy="0 0 0"/>
-            <geometry>
-                <box size="${camera_size_x} ${camera_size_y} ${camera_size_z}"/>
-            </geometry>
+            <geometry><box size="0.040 0.025 0.025"/></geometry>
         </collision>
         <inertial>
             <mass value="${camera_mass}"/>
             <origin xyz="0 0 0" rpy="0 0 0"/>
-            <inertia
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