Commit message: feat(urdf): replace primitive arm with official SO-101 STL mesh model
- Download all 13 official STL assets from TheRobotStudio/SO-ARM100
  into robot_ws/src/omnibot_description/meshes/so101/
- Replace every arm link visual/collision from box+cylinder primitives
  to exact mesh geometry from so101_new_calib.urdf (onshape-to-robot)
- Preserve ALL official joint origins, axes, and limits verbatim
- Add arm_gripper_frame_link (tool-frame reference, fixed joint)
- Rename arm_jaw_link → arm_moving_jaw_link to match official naming
- Transmissions renamed to arm_motor1..6 matching official actuator IDs
- Meshes referenced via package://omnibot_description/meshes/so101/

Co-Authored-By: Claude Sonnet 4.6 <noreply@anthropic.com>

File: robot_ws/src/omnibot_description/urdf/omnibot.urdf.xacro (robot description, xacro)
@@ -534,50 +534,15 @@
     <xacro:wheel prefix="rear_right"  x_reflect="-1" y_reflect="-1" cs=" 1"/>
     <!-- ================================================================
-         SO-ARM 101  — 6-DOF serial arm mounted at the FRONT of the
-         top plate, centred left-to-right.
-         Links use simplified box/cylinder primitives (no STL meshes).
-         Joint kinematics match the official so101_new_calib.urdf from
-         TheRobotStudio/SO-ARM100 (joint origins & limits preserved).
-         Link colours:
-           White  (1 1 1 1)  — 3D-printed PLA parts
-           Dark   (0.15 0.15 0.15 1) — STS3215 servo bodies
-         Arm is mounted at x=+0.055 m (front area) in top_plate frame.
-         ================================================================ -->
-    <!-- ARM BASE — servo pedestal + WaveShare mounting plate -->
-    <link name="arm_base_link">
-        <visual>
-            <origin xyz="0 0 0.031" rpy="0 0 0"/>
-            <geometry>
-                <box size="0.075 0.075 0.062"/>
-            </geometry>
-            <material name="arm_white">
-                <color rgba="0.95 0.95 0.95 1"/>
-            </material>
-        </visual>
-        <!-- Bottom servo body (dark) -->
-        <visual>
-            <origin xyz="0.026 0 0.044" rpy="0 0 0"/>
-            <geometry>
-                <box size="0.040 0.025 0.040"/>
-            </geometry>
-            <material name="servo_dark">
-                <color rgba="0.15 0.15 0.15 1"/>
-            </material>
-        </visual>
-        <collision>
-            <origin xyz="0 0 0.031" rpy="0 0 0"/>
-            <geometry>
-                <box size="0.075 0.075 0.062"/>
-            </geometry>
-        </collision>
-        <inertial>
-            <mass value="0.147"/>
-            <origin xyz="0 0 0.031" rpy="0 0 0"/>
-            <inertia ixx="0.000115" ixy="0" ixz="0"
-                     iyy="0.000136" iyz="0"
-                     izz="0.000130"/>
-        </inertial>
-    </link>
-    <!-- Arm sits at the front of the top plate, on its top surface -->
+         SO-ARM 101 — Official 6-DOF follower arm
+         Source: TheRobotStudio/SO-ARM100  Simulation/SO101/so101_new_calib.urdf
+         STL meshes: package://omnibot_description/meshes/so101/
+         All joint origins, axes, and limits are EXACT from the official URDF.
+         Link names prefixed with "arm_" to avoid collisions with robot links.
+         Arm base mounted at the FRONT-CENTRE of the top plate.
+         ================================================================ -->
+    <!-- Arm materials -->
+    <material name="arm_3d_printed"><color rgba="1.0 1.0 1.0 1.0"/></material>
+    <material name="arm_sts3215"><color rgba="0.1 0.1 0.1 1.0"/></material>
+    <!-- Fixed joint: top plate → arm base (front-centre of top plate) -->
     <joint name="arm_base_joint" type="fixed">
         <parent link="top_plate_link"/>
@@ -585,41 +550,89 @@
         <origin xyz="0.055 0 ${plate_thickness / 2.0}" rpy="0 0 0"/>
     </joint>
-    <!-- SHOULDER — pan joint (rotates about Z, vertical axis) -->
+    <!-- ARM BASE LINK (base_motor_holder + base plate + servo + waveshare mount) -->
+    <link name="arm_base_link">
+        <inertial>
+            <origin xyz="0.0137179 -5.19711e-05 0.0334843" rpy="0 0 0"/>
+            <mass value="0.147"/>
+            <inertia ixx="0.000114686" ixy="-4.59787e-07" ixz="4.97151e-06"
+                     iyy="0.000136117" iyz="9.75275e-08" izz="0.000130364"/>
+        </inertial>
+        <visual>
+            <origin xyz="-0.00636471 -9.94414e-05 -0.0024" rpy="1.5708 -1.67685e-15 1.5708"/>
+            <geometry><mesh filename="package://omnibot_description/meshes/so101/base_motor_holder_so101_v1.stl"/></geometry>
+            <material name="arm_3d_printed"/>
+        </visual>
+        <collision>
+            <origin xyz="-0.00636471 -9.94414e-05 -0.0024" rpy="1.5708 -1.67685e-15 1.5708"/>
+            <geometry><mesh filename="package://omnibot_description/meshes/so101/base_motor_holder_so101_v1.stl"/></geometry>
+        </collision>
+        <visual>
+            <origin xyz="-0.00636471 -8.97657e-09 -0.0024" rpy="1.5708 -2.78073e-29 1.5708"/>
+            <geometry><mesh filename="package://omnibot_description/meshes/so101/base_so101_v2.stl"/></geometry>
+            <material name="arm_3d_printed"/>
+        </visual>
+        <collision>
+            <origin xyz="-0.00636471 -8.97657e-09 -0.0024" rpy="1.5708 -2.78073e-29 1.5708"/>
+            <geometry><mesh filename="package://omnibot_description/meshes/so101/base_so101_v2.stl"/></geometry>
+        </collision>
+        <visual>
+            <origin xyz="0.0263353 -8.97657e-09 0.0437" rpy="-8.21148e-16 7.84513e-18 1.249e-15"/>
+            <geometry><mesh filename="package://omnibot_description/meshes/so101/sts3215_03a_v1.stl"/></geometry>
+            <material name="arm_sts3215"/>
+        </visual>
+        <collision>
+            <origin xyz="0.0263353 -8.97657e-09 0.0437" rpy="-8.21148e-16 7.84513e-18 1.249e-15"/>
+            <geometry><mesh filename="package://omnibot_description/meshes/so101/sts3215_03a_v1.stl"/></geometry>
+        </collision>
+        <visual>
+            <origin xyz="-0.0309827 -0.000199441 0.0474" rpy="1.5708 -1.35493e-14 1.5708"/>
+            <geometry><mesh filename="package://omnibot_description/meshes/so101/waveshare_mounting_plate_so101_v2.stl"/></geometry>
+            <material name="arm_3d_printed"/>
+        </visual>
+        <collision>
+            <origin xyz="-0.0309827 -0.000199441 0.0474" rpy="1.5708 -1.35493e-14 1.5708"/>
+            <geometry><mesh filename="package://omnibot_description/meshes/so101/waveshare_mounting_plate_so101_v2.stl"/></geometry>
+        </collision>
+    </link>
+    <!-- SHOULDER LINK (sts3215 servo + motor_holder_base + rotation_pitch) -->
     <link name="arm_shoulder_link">
-        <!-- Shoulder servo (dark) -->
-        <visual>
-            <origin xyz="-0.030 0 -0.025" rpy="${PI/2} 0 0"/>
-            <geometry>
-                <cylinder radius="0.020" length="0.050"/>
-            </geometry>
-            <material name="servo_dark"/>
-        </visual>
-        <!-- Motor holder + rotation pitch bracket (white) -->
-        <visual>
-            <origin xyz="0.012 0 0.046" rpy="0 0 0"/>
-            <geometry>
-                <box size="0.040 0.045 0.035"/>
-            </geometry>
-            <material name="arm_white"/>
-        </visual>
-        <collision>
-            <origin xyz="-0.030 0 -0.025" rpy="${PI/2} 0 0"/>
-            <geometry>
-                <cylinder radius="0.020" length="0.050"/>
-            </geometry>
-        </collision>
-        <inertial>
-            <mass value="0.100"/>
-            <origin xyz="-0.031 0 -0.025" rpy="0 0 0"/>
-            <inertia ixx="8.4e-05" ixy="0" ixz="0"
-                     iyy="8.1e-05" iyz="0"
-                     izz="2.4e-05"/>
-        </inertial>
-    </link>
-    <!-- shoulder_pan: origin from SO-101 official URDF -->
+        <inertial>
+            <origin xyz="-0.0307604 -1.66727e-05 -0.0252713" rpy="0 0 0"/>
+            <mass value="0.100006"/>
+            <inertia ixx="8.3759e-05" ixy="7.55525e-08" ixz="-1.16342e-06"
+                     iyy="8.10403e-05" iyz="1.54663e-07" izz="2.39783e-05"/>
+        </inertial>
+        <visual>
+            <origin xyz="-0.0303992 0.000422241 -0.0417" rpy="1.5708 1.5708 0"/>
+            <geometry><mesh filename="package://omnibot_description/meshes/so101/sts3215_03a_v1.stl"/></geometry>
+            <material name="arm_sts3215"/>
+        </visual>
+        <collision>
+            <origin xyz="-0.0303992 0.000422241 -0.0417" rpy="1.5708 1.5708 0"/>
+            <geometry><mesh filename="package://omnibot_description/meshes/so101/sts3215_03a_v1.stl"/></geometry>
+        </collision>
+        <visual>
+            <origin xyz="-0.0675992 -0.000177759 0.0158499" rpy="1.5708 -1.5708 0"/>
+            <geometry><mesh filename="package://omnibot_description/meshes/so101/motor_holder_so101_base_v1.stl"/></geometry>
+            <material name="arm_3d_printed"/>
+        </visual>
+        <collision>
+            <origin xyz="-0.0675992 -0.000177759 0.0158499" rpy="1.5708 -1.5708 0"/>
+            <geometry><mesh filename="package://omnibot_description/meshes/so101/motor_holder_so101_base_v1.stl"/></geometry>
+        </collision>
+        <visual>
+            <origin xyz="0.0122008 2.22413e-05 0.0464" rpy="-1.5708 2.35221e-33 0"/>
+            <geometry><mesh filename="package://omnibot_description/meshes/so101/rotation_pitch_so101_v1.stl"/></geometry>
+            <material name="arm_3d_printed"/>
+        </visual>
+        <collision>
+            <origin xyz="0.0122008 2.22413e-05 0.0464" rpy="-1.5708 2.35221e-33 0"/>
+            <geometry><mesh filename="package://omnibot_description/meshes/so101/rotation_pitch_so101_v1.stl"/></geometry>
+        </collision>
+    </link>
     <joint name="arm_shoulder_pan" type="revolute">
+        <origin xyz="0.0388353 -8.97657e-09 0.0624" rpy="3.14159 4.18253e-17 -3.14159"/>
         <parent link="arm_base_link"/>
         <child link="arm_shoulder_link"/>
-        <origin xyz="0.0388353 0 0.0624" rpy="${PI} 0 ${-PI}"/>
         <axis xyz="0 0 1"/>
         <limit effort="10" velocity="10" lower="-1.91986" upper="1.91986"/>
@@ -630,46 +643,40 @@
             <hardwareInterface>hardware_interface/PositionJointInterface</hardwareInterface>
         </joint>
-        <actuator name="arm_shoulder_pan_motor">
+        <actuator name="arm_motor1">
             <hardwareInterface>hardware_interface/PositionJointInterface</hardwareInterface>
             <mechanicalReduction>1</mechanicalReduction>
         </actuator>
     </transmission>
-    <!-- UPPER ARM -->
+    <!-- UPPER ARM LINK (upper_arm + sts3215 elbow servo) -->
     <link name="arm_upper_arm_link">
-        <!-- Upper arm beam (white) -->
-        <visual>
-            <origin xyz="-0.065 0.012 0.018" rpy="0 0 0"/>
-            <geometry>
-                <box size="0.125 0.035 0.030"/>
-            </geometry>
-            <material name="arm_white"/>
-        </visual>
-        <!-- Elbow servo (dark) -->
-        <visual>
-            <origin xyz="-0.113 -0.016 0.019" rpy="${-PI} 0 ${-PI/2}"/>
-            <geometry>
-                <cylinder radius="0.018" length="0.040"/>
-            </geometry>
-            <material name="servo_dark"/>
-        </visual>
-        <collision>
-            <origin xyz="-0.065 0.012 0.018" rpy="0 0 0"/>
-            <geometry>
-                <box size="0.125 0.035 0.030"/>
-            </geometry>
-        </collision>
-        <inertial>
+        <inertial>
+            <origin xyz="-0.0898471 -0.00838224 0.0184089" rpy="0 0 0"/>
             <mass value="0.103"/>
-            <origin xyz="-0.090 -0.008 0.018" rpy="0 0 0"/>
-            <inertia ixx="4.1e-05" ixy="-2.0e-05" ixz="0"
-                     iyy="1.47e-04" iyz="0"
-                     izz="1.42e-04"/>
-        </inertial>
-    </link>
-    <!-- shoulder_lift: origin from SO-101 official URDF -->
+            <inertia ixx="4.08002e-05" ixy="-1.97819e-05" ixz="-4.03016e-08"
+                     iyy="0.000147318" iyz="8.97326e-09" izz="0.000142487"/>
+        </inertial>
+        <visual>
+            <origin xyz="-0.11257 -0.0155 0.0187" rpy="-3.14159 -5.27356e-16 -1.5708"/>
+            <geometry><mesh filename="package://omnibot_description/meshes/so101/sts3215_03a_v1.stl"/></geometry>
+            <material name="arm_sts3215"/>
+        </visual>
+        <collision>
+            <origin xyz="-0.11257 -0.0155 0.0187" rpy="-3.14159 -5.27356e-16 -1.5708"/>
+            <geometry><mesh filename="package://omnibot_description/meshes/so101/sts3215_03a_v1.stl"/></geometry>
+        </collision>
+        <visual>
+            <origin xyz="-0.065085 0.012 0.0182" rpy="3.14159 -0 -1.30911e-30"/>
+            <geometry><mesh filename="package://omnibot_description/meshes/so101/upper_arm_so101_v1.stl"/></geometry>
+            <material name="arm_3d_printed"/>
+        </visual>
+        <collision>
+            <origin xyz="-0.065085 0.012 0.0182" rpy="3.14159 -0 -1.30911e-30"/>
+            <geometry><mesh filename="package://omnibot_description/meshes/so101/upper_arm_so101_v1.stl"/></geometry>
+        </collision>
+    </link>
     <joint name="arm_shoulder_lift" type="revolute">
+        <origin xyz="-0.0303992 -0.0182778 -0.0542" rpy="-1.5708 -1.5708 0"/>
         <parent link="arm_shoulder_link"/>
         <child link="arm_upper_arm_link"/>
-        <origin xyz="-0.0303992 -0.0182778 -0.0542" rpy="${-PI/2} ${-PI/2} 0"/>
         <axis xyz="0 0 1"/>
         <limit effort="10" velocity="10" lower="-1.74533" upper="1.74533"/>
@@ -680,46 +687,49 @@
             <hardwareInterface>hardware_interface/PositionJointInterface</hardwareInterface>
         </joint>
-        <actuator name="arm_shoulder_lift_motor">
+        <actuator name="arm_motor2">
             <hardwareInterface>hardware_interface/PositionJointInterface</hardwareInterface>
             <mechanicalReduction>1</mechanicalReduction>
         </actuator>
     </transmission>
-    <!-- LOWER ARM (forearm) -->
+    <!-- LOWER ARM LINK (under_arm + motor_holder_wrist + sts3215 wrist servo) -->
     <link name="arm_lower_arm_link">
-        <!-- Forearm beam (white) -->
-        <visual>
-            <origin xyz="-0.065 -0.032 0.018" rpy="0 0 0"/>
-            <geometry>
-                <box size="0.125 0.030 0.028"/>
-            </geometry>
-            <material name="arm_white"/>
-        </visual>
-        <!-- Wrist servo (dark) -->
-        <visual>
-            <origin xyz="-0.122 0.005 0.019" rpy="${-PI} 0 ${-PI}"/>
-            <geometry>
-                <cylinder radius="0.018" length="0.040"/>
-            </geometry>
-            <material name="servo_dark"/>
-        </visual>
-        <collision>
-            <origin xyz="-0.065 -0.032 0.018" rpy="0 0 0"/>
-            <geometry>
-                <box size="0.125 0.030 0.028"/>
-            </geometry>
-        </collision>
-        <inertial>
+        <inertial>
+            <origin xyz="-0.0980701 0.00324376 0.0182831" rpy="0 0 0"/>
             <mass value="0.104"/>
-            <origin xyz="-0.098 0.003 0.018" rpy="0 0 0"/>
-            <inertia ixx="2.9e-05" ixy="7.4e-06" ixz="0"
-                     iyy="1.60e-04" iyz="0"
-                     izz="1.45e-04"/>
-        </inertial>
-    </link>
-    <!-- elbow_flex: origin from SO-101 official URDF -->
+            <inertia ixx="2.87438e-05" ixy="7.41152e-06" ixz="1.26409e-06"
+                     iyy="0.000159844" iyz="-4.90188e-08" izz="0.00014529"/>
+        </inertial>
+        <visual>
+            <origin xyz="-0.0648499 -0.032 0.0182" rpy="3.14159 -0 6.67202e-31"/>
+            <geometry><mesh filename="package://omnibot_description/meshes/so101/under_arm_so101_v1.stl"/></geometry>
+            <material name="arm_3d_printed"/>
+        </visual>
+        <collision>
+            <origin xyz="-0.0648499 -0.032 0.0182" rpy="3.14159 -0 6.67202e-31"/>
+            <geometry><mesh filename="package://omnibot_description/meshes/so101/under_arm_so101_v1.stl"/></geometry>
+        </collision>
+        <visual>
+            <origin xyz="-0.0648499 -0.032 0.018" rpy="-3.14159 -2.55351e-15 -1.83387e-30"/>
+            <geometry><mesh filename="package://omnibot_description/meshes/so101/motor_holder_so101_wrist_v1.stl"/></geometry>
+            <material name="arm_3d_printed"/>
+        </visual>
+        <collision>
+            <origin xyz="-0.0648499 -0.032 0.018" rpy="-3.14159 -2.55351e-15 -1.83387e-30"/>
+            <geometry><mesh filename="package://omnibot_description/meshes/so101/motor_holder_so101_wrist_v1.stl"/></geometry>
+        </collision>
+        <visual>
+            <origin xyz="-0.1224 0.0052 0.0187" rpy="-3.14159 -7.88861e-31 -3.14159"/>
+            <geometry><mesh filename="package://omnibot_description/meshes/so101/sts3215_03a_v1.stl"/></geometry>
+            <material name="arm_sts3215"/>
+        </visual>
+        <collision>
+            <origin xyz="-0.1224 0.0052 0.0187" rpy="-3.14159 -7.88861e-31 -3.14159"/>
+            <geometry><mesh filename="package://omnibot_description/meshes/so101/sts3215_03a_v1.stl"/></geometry>
+        </collision>
+    </link>
     <joint name="arm_elbow_flex" type="revolute">
+        <origin xyz="-0.11257 -0.028 1.73763e-16" rpy="-3.63608e-16 8.74301e-16 1.5708"/>
         <parent link="arm_upper_arm_link"/>
         <child link="arm_lower_arm_link"/>
-        <origin xyz="-0.11257 -0.028 0" rpy="0 0 ${PI/2}"/>
         <axis xyz="0 0 1"/>
         <limit effort="10" velocity="10" lower="-1.69" upper="1.69"/>
@@ -730,46 +740,40 @@
             <hardwareInterface>hardware_interface/PositionJointInterface</hardwareInterface>
         </joint>
-        <actuator name="arm_elbow_flex_motor">
+        <actuator name="arm_motor3">
             <hardwareInterface>hardware_interface/PositionJointInterface</hardwareInterface>
             <mechanicalReduction>1</mechanicalReduction>
         </actuator>
     </transmission>
-    <!-- WRIST -->
+    <!-- WRIST LINK (wrist_roll_pitch + sts3215_no_horn) -->
     <link name="arm_wrist_link">
-        <!-- Wrist roll servo (dark) -->
-        <visual>
-            <origin xyz="0 -0.042 0.031" rpy="${PI/2} ${PI/2} 0"/>
-            <geometry>
-                <cylinder radius="0.018" length="0.040"/>
-            </geometry>
-            <material name="servo_dark"/>
-        </visual>
-        <!-- Wrist body (white) -->
-        <visual>
-            <origin xyz="0 -0.028 0.018" rpy="0 0 0"/>
-            <geometry>
-                <box size="0.038 0.035 0.035"/>
-            </geometry>
-            <material name="arm_white"/>
-        </visual>
-        <collision>
-            <origin xyz="0 -0.028 0.018" rpy="0 0 0"/>
-            <geometry>
-                <box size="0.038 0.035 0.035"/>
-            </geometry>
-        </collision>
-        <inertial>
-            <mass value="0.060"/>
-            <origin xyz="0 -0.039 0.028" rpy="0 0 0"/>
-            <inertia ixx="5.0e-05" ixy="0" ixz="0"
-                     iyy="4.0e-05" iyz="0"
-                     izz="3.0e-05"/>
-        </inertial>
-    </link>
-    <!-- wrist_flex: origin from SO-101 official URDF -->
+        <inertial>
+            <origin xyz="-0.000103312 -0.0386143 0.0281156" rpy="0 0 0"/>
+            <mass value="0.079"/>
+            <inertia ixx="3.68263e-05" ixy="1.7893e-08" ixz="-5.28128e-08"
+                     iyy="2.5391e-05" iyz="3.6412e-06" izz="2.1e-05"/>
+        </inertial>
+        <visual>
+            <origin xyz="8.32667e-17 -0.0424 0.0306" rpy="1.5708 1.5708 0"/>
+            <geometry><mesh filename="package://omnibot_description/meshes/so101/sts3215_03a_no_horn_v1.stl"/></geometry>
+            <material name="arm_sts3215"/>
+        </visual>
+        <collision>
+            <origin xyz="8.32667e-17 -0.0424 0.0306" rpy="1.5708 1.5708 0"/>
+            <geometry><mesh filename="package://omnibot_description/meshes/so101/sts3215_03a_no_horn_v1.stl"/></geometry>
+        </collision>
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