Commit message: fix(urdf): revert arm visuals to primitives, add mecanum rollers, integrate SO-101 structure
- Arm link visuals changed from STL mesh (package://) to box/cylinder primitives
  so the URDF renders in any viewer without colcon build
- All 6 revolute + 1 fixed SO-ARM 101 joint origins/axes/limits preserved exactly
  from the official so101_new_calib.urdf (TheRobotStudio/SO-ARM100)
- STL mesh files kept in meshes/so101/ for future ROS 2 deployment
- Mecanum wheel macro: removed incorrect yaw, added 8 barrel rollers per wheel
  with analytically derived 45-degree diagonal orientations
- gripper_frame_link inertia set to 1e-9 (was 0, which is singular)
- Removed invalid <axis> from fixed joint arm_gripper_frame_joint

Co-Authored-By: Claude Sonnet 4.6 <noreply@anthropic.com>

File: robot_ws/src/omnibot_description/urdf/omnibot.urdf.xacro (robot description, xacro)
@@ -534,15 +534,12 @@
     <xacro:wheel prefix="rear_right"  x_reflect="-1" y_reflect="-1" cs=" 1"/>
     <!-- ================================================================
-         SO-ARM 101 — Official 6-DOF follower arm
-         Source: TheRobotStudio/SO-ARM100  Simulation/SO101/so101_new_calib.urdf
-         STL meshes: package://omnibot_description/meshes/so101/
-         All joint origins, axes, and limits are EXACT from the official URDF.
-         Link names prefixed with "arm_" to avoid collisions with robot links.
-         Arm base mounted at the FRONT-CENTRE of the top plate.
-         ================================================================ -->
-    <!-- Arm materials -->
-    <material name="arm_3d_printed"><color rgba="1.0 1.0 1.0 1.0"/></material>
-    <material name="arm_sts3215"><color rgba="0.1 0.1 0.1 1.0"/></material>
-    <!-- Fixed joint: top plate → arm base (front-centre of top plate) -->
+         SO-ARM 101 — 6-DOF follower arm (TheRobotStudio/SO-ARM100)
+         Joint origins/axes/limits: EXACT from so101_new_calib.urdf.
+         Visuals: box + cylinder primitives (render in any viewer).
+         STL meshes kept in meshes/so101/ for ROS 2 use after colcon build.
+         ================================================================ -->
+    <material name="arm_white"><color rgba="0.95 0.95 0.95 1.0"/></material>
+    <material name="arm_servo"><color rgba="0.12 0.12 0.12 1.0"/></material>
+    <!-- Fixed joint: top plate → arm base -->
     <joint name="arm_base_joint" type="fixed">
         <parent link="top_plate_link"/>
@@ -550,6 +547,28 @@
         <origin xyz="0.055 0 ${plate_thickness / 2.0}" rpy="0 0 0"/>
     </joint>
-    <!-- ARM BASE LINK (base_motor_holder + base plate + servo + waveshare mount) -->
+    <!-- ARM BASE — pedestal body + bottom servo -->
     <link name="arm_base_link">
+        <visual>
+            <!-- Main body: ~75×65×55 mm box, centred at z=0.035 -->
+            <origin xyz="0 0 0.035" rpy="0 0 0"/>
+            <geometry><box size="0.075 0.065 0.055"/></geometry>
+            <material name="arm_white"/>
+        </visual>
+        <visual>
+            <!-- STS3215 base servo body -->
+            <origin xyz="0.026 0 0.044" rpy="0 0 0"/>
+            <geometry><box size="0.040 0.025 0.040"/></geometry>
+            <material name="arm_servo"/>
+        </visual>
+        <visual>
+            <!-- Waveshare mounting plate on top -->
+            <origin xyz="-0.031 0 0.068" rpy="0 0 0"/>
+            <geometry><box size="0.080 0.060 0.006"/></geometry>
+            <material name="arm_white"/>
+        </visual>
+        <collision>
+            <origin xyz="0 0 0.035" rpy="0 0 0"/>
+            <geometry><box size="0.075 0.065 0.070"/></geometry>
+        </collision>
         <inertial>
             <origin xyz="0.0137179 -5.19711e-05 0.0334843" rpy="0 0 0"/>
@@ -558,43 +577,23 @@
                      iyy="0.000136117" iyz="9.75275e-08" izz="0.000130364"/>
         </inertial>
-        <visual>
-            <origin xyz="-0.00636471 -9.94414e-05 -0.0024" rpy="1.5708 -1.67685e-15 1.5708"/>
-            <geometry><mesh filename="package://omnibot_description/meshes/so101/base_motor_holder_so101_v1.stl"/></geometry>
-            <material name="arm_3d_printed"/>
-        </visual>
-        <collision>
-            <origin xyz="-0.00636471 -9.94414e-05 -0.0024" rpy="1.5708 -1.67685e-15 1.5708"/>
-            <geometry><mesh filename="package://omnibot_description/meshes/so101/base_motor_holder_so101_v1.stl"/></geometry>
-        </collision>
-        <visual>
-            <origin xyz="-0.00636471 -8.97657e-09 -0.0024" rpy="1.5708 -2.78073e-29 1.5708"/>
-            <geometry><mesh filename="package://omnibot_description/meshes/so101/base_so101_v2.stl"/></geometry>
-            <material name="arm_3d_printed"/>
-        </visual>
-        <collision>
-            <origin xyz="-0.00636471 -8.97657e-09 -0.0024" rpy="1.5708 -2.78073e-29 1.5708"/>
-            <geometry><mesh filename="package://omnibot_description/meshes/so101/base_so101_v2.stl"/></geometry>
-        </collision>
-        <visual>
-            <origin xyz="0.0263353 -8.97657e-09 0.0437" rpy="-8.21148e-16 7.84513e-18 1.249e-15"/>
-            <geometry><mesh filename="package://omnibot_description/meshes/so101/sts3215_03a_v1.stl"/></geometry>
-            <material name="arm_sts3215"/>
-        </visual>
-        <collision>
-            <origin xyz="0.0263353 -8.97657e-09 0.0437" rpy="-8.21148e-16 7.84513e-18 1.249e-15"/>
-            <geometry><mesh filename="package://omnibot_description/meshes/so101/sts3215_03a_v1.stl"/></geometry>
-        </collision>
-        <visual>
-            <origin xyz="-0.0309827 -0.000199441 0.0474" rpy="1.5708 -1.35493e-14 1.5708"/>
-            <geometry><mesh filename="package://omnibot_description/meshes/so101/waveshare_mounting_plate_so101_v2.stl"/></geometry>
-            <material name="arm_3d_printed"/>
-        </visual>
-        <collision>
-            <origin xyz="-0.0309827 -0.000199441 0.0474" rpy="1.5708 -1.35493e-14 1.5708"/>
-            <geometry><mesh filename="package://omnibot_description/meshes/so101/waveshare_mounting_plate_so101_v2.stl"/></geometry>
-        </collision>
-    </link>
-    <!-- SHOULDER LINK (sts3215 servo + motor_holder_base + rotation_pitch) -->
+    </link>
+    <!-- SHOULDER — pan servo + motor holder + rotation pitch bracket -->
     <link name="arm_shoulder_link">
+        <visual>
+            <!-- STS3215 shoulder servo, lying on its side -->
+            <origin xyz="-0.031 0 -0.025" rpy="${PI/2} 0 0"/>
+            <geometry><cylinder radius="0.020" length="0.050"/></geometry>
+            <material name="arm_servo"/>
+        </visual>
+        <visual>
+            <!-- Motor holder + rotation pitch bracket -->
+            <origin xyz="0.012 0 0.046" rpy="0 0 0"/>
+            <geometry><box size="0.040 0.045 0.038"/></geometry>
+            <material name="arm_white"/>
+        </visual>
+        <collision>
+            <origin xyz="-0.031 0 -0.025" rpy="${PI/2} 0 0"/>
+            <geometry><cylinder radius="0.020" length="0.050"/></geometry>
+        </collision>
         <inertial>
             <origin xyz="-0.0307604 -1.66727e-05 -0.0252713" rpy="0 0 0"/>
@@ -603,32 +602,6 @@
                      iyy="8.10403e-05" iyz="1.54663e-07" izz="2.39783e-05"/>
         </inertial>
-        <visual>
-            <origin xyz="-0.0303992 0.000422241 -0.0417" rpy="1.5708 1.5708 0"/>
-            <geometry><mesh filename="package://omnibot_description/meshes/so101/sts3215_03a_v1.stl"/></geometry>
-            <material name="arm_sts3215"/>
-        </visual>
-        <collision>
-            <origin xyz="-0.0303992 0.000422241 -0.0417" rpy="1.5708 1.5708 0"/>
-            <geometry><mesh filename="package://omnibot_description/meshes/so101/sts3215_03a_v1.stl"/></geometry>
-        </collision>
-        <visual>
-            <origin xyz="-0.0675992 -0.000177759 0.0158499" rpy="1.5708 -1.5708 0"/>
-            <geometry><mesh filename="package://omnibot_description/meshes/so101/motor_holder_so101_base_v1.stl"/></geometry>
-            <material name="arm_3d_printed"/>
-        </visual>
-        <collision>
-            <origin xyz="-0.0675992 -0.000177759 0.0158499" rpy="1.5708 -1.5708 0"/>
-            <geometry><mesh filename="package://omnibot_description/meshes/so101/motor_holder_so101_base_v1.stl"/></geometry>
-        </collision>
-        <visual>
-            <origin xyz="0.0122008 2.22413e-05 0.0464" rpy="-1.5708 2.35221e-33 0"/>
-            <geometry><mesh filename="package://omnibot_description/meshes/so101/rotation_pitch_so101_v1.stl"/></geometry>
-            <material name="arm_3d_printed"/>
-        </visual>
-        <collision>
-            <origin xyz="0.0122008 2.22413e-05 0.0464" rpy="-1.5708 2.35221e-33 0"/>
-            <geometry><mesh filename="package://omnibot_description/meshes/so101/rotation_pitch_so101_v1.stl"/></geometry>
-        </collision>
-    </link>
+    </link>
+    <!-- shoulder_pan — exact origin from so101_new_calib.urdf -->
     <joint name="arm_shoulder_pan" type="revolute">
         <origin xyz="0.0388353 -8.97657e-09 0.0624" rpy="3.14159 4.18253e-17 -3.14159"/>
@@ -648,6 +621,22 @@
         </actuator>
     </transmission>
-    <!-- UPPER ARM LINK (upper_arm + sts3215 elbow servo) -->
+    <!-- UPPER ARM — beam + elbow servo -->
     <link name="arm_upper_arm_link">
+        <visual>
+            <!-- Upper arm beam -->
+            <origin xyz="-0.065 0.012 0.018" rpy="0 0 0"/>
+            <geometry><box size="0.125 0.035 0.030"/></geometry>
+            <material name="arm_white"/>
+        </visual>
+        <visual>
+            <!-- STS3215 elbow servo -->
+            <origin xyz="-0.113 -0.016 0.019" rpy="${PI/2} 0 0"/>
+            <geometry><cylinder radius="0.018" length="0.040"/></geometry>
+            <material name="arm_servo"/>
+        </visual>
+        <collision>
+            <origin xyz="-0.065 0.012 0.018" rpy="0 0 0"/>
+            <geometry><box size="0.125 0.035 0.030"/></geometry>
+        </collision>
         <inertial>
             <origin xyz="-0.0898471 -0.00838224 0.0184089" rpy="0 0 0"/>
@@ -656,23 +645,6 @@
                      iyy="0.000147318" iyz="8.97326e-09" izz="0.000142487"/>
         </inertial>
-        <visual>
-            <origin xyz="-0.11257 -0.0155 0.0187" rpy="-3.14159 -5.27356e-16 -1.5708"/>
-            <geometry><mesh filename="package://omnibot_description/meshes/so101/sts3215_03a_v1.stl"/></geometry>
-            <material name="arm_sts3215"/>
-        </visual>
-        <collision>
-            <origin xyz="-0.11257 -0.0155 0.0187" rpy="-3.14159 -5.27356e-16 -1.5708"/>
-            <geometry><mesh filename="package://omnibot_description/meshes/so101/sts3215_03a_v1.stl"/></geometry>
-        </collision>
-        <visual>
-            <origin xyz="-0.065085 0.012 0.0182" rpy="3.14159 -0 -1.30911e-30"/>
-            <geometry><mesh filename="package://omnibot_description/meshes/so101/upper_arm_so101_v1.stl"/></geometry>
-            <material name="arm_3d_printed"/>
-        </visual>
-        <collision>
-            <origin xyz="-0.065085 0.012 0.0182" rpy="3.14159 -0 -1.30911e-30"/>
-            <geometry><mesh filename="package://omnibot_description/meshes/so101/upper_arm_so101_v1.stl"/></geometry>
-        </collision>
-    </link>
+    </link>
+    <!-- shoulder_lift — exact origin from so101_new_calib.urdf -->
     <joint name="arm_shoulder_lift" type="revolute">
         <origin xyz="-0.0303992 -0.0182778 -0.0542" rpy="-1.5708 -1.5708 0"/>
@@ -692,6 +664,22 @@
         </actuator>
     </transmission>
-    <!-- LOWER ARM LINK (under_arm + motor_holder_wrist + sts3215 wrist servo) -->
+    <!-- LOWER ARM — forearm beam + wrist servo -->
     <link name="arm_lower_arm_link">
+        <visual>
+            <!-- Forearm beam -->
+            <origin xyz="-0.065 -0.032 0.018" rpy="0 0 0"/>
+            <geometry><box size="0.125 0.030 0.028"/></geometry>
+            <material name="arm_white"/>
+        </visual>
+        <visual>
+            <!-- STS3215 wrist servo -->
+            <origin xyz="-0.122 0.005 0.019" rpy="${PI/2} 0 0"/>
+            <geometry><cylinder radius="0.018" length="0.040"/></geometry>
+            <material name="arm_servo"/>
+        </visual>
+        <collision>
+            <origin xyz="-0.065 -0.032 0.018" rpy="0 0 0"/>
+            <geometry><box size="0.125 0.030 0.028"/></geometry>
+        </collision>
         <inertial>
             <origin xyz="-0.0980701 0.00324376 0.0182831" rpy="0 0 0"/>
@@ -700,32 +688,6 @@
                      iyy="0.000159844" iyz="-4.90188e-08" izz="0.00014529"/>
         </inertial>
-        <visual>
-            <origin xyz="-0.0648499 -0.032 0.0182" rpy="3.14159 -0 6.67202e-31"/>
-            <geometry><mesh filename="package://omnibot_description/meshes/so101/under_arm_so101_v1.stl"/></geometry>
-            <material name="arm_3d_printed"/>
-        </visual>
-        <collision>
-            <origin xyz="-0.0648499 -0.032 0.0182" rpy="3.14159 -0 6.67202e-31"/>
-            <geometry><mesh filename="package://omnibot_description/meshes/so101/under_arm_so101_v1.stl"/></geometry>
-        </collision>
-        <visual>
-            <origin xyz="-0.0648499 -0.032 0.018" rpy="-3.14159 -2.55351e-15 -1.83387e-30"/>
-            <geometry><mesh filename="package://omnibot_description/meshes/so101/motor_holder_so101_wrist_v1.stl"/></geometry>
-            <material name="arm_3d_printed"/>
-        </visual>
-        <collision>
-            <origin xyz="-0.0648499 -0.032 0.018" rpy="-3.14159 -2.55351e-15 -1.83387e-30"/>
-            <geometry><mesh filename="package://omnibot_description/meshes/so101/motor_holder_so101_wrist_v1.stl"/></geometry>
-        </collision>
-        <visual>
-            <origin xyz="-0.1224 0.0052 0.0187" rpy="-3.14159 -7.88861e-31 -3.14159"/>
-            <geometry><mesh filename="package://omnibot_description/meshes/so101/sts3215_03a_v1.stl"/></geometry>
-            <material name="arm_sts3215"/>
-        </visual>
-        <collision>
-            <origin xyz="-0.1224 0.0052 0.0187" rpy="-3.14159 -7.88861e-31 -3.14159"/>
-            <geometry><mesh filename="package://omnibot_description/meshes/so101/sts3215_03a_v1.stl"/></geometry>
-        </collision>
-    </link>
+    </link>
+    <!-- elbow_flex — exact origin from so101_new_calib.urdf -->
     <joint name="arm_elbow_flex" type="revolute">
         <origin xyz="-0.11257 -0.028 1.73763e-16" rpy="-3.63608e-16 8.74301e-16 1.5708"/>
@@ -745,6 +707,22 @@
         </actuator>
     </transmission>
-    <!-- WRIST LINK (wrist_roll_pitch + sts3215_no_horn) -->
+    <!-- WRIST — roll/pitch bracket + servo (no horn) -->
     <link name="arm_wrist_link">
+        <visual>
+            <!-- Wrist roll-pitch body -->
+            <origin xyz="0 -0.028 0.018" rpy="0 0 0"/>
+            <geometry><box size="0.038 0.035 0.040"/></geometry>
+            <material name="arm_white"/>
+        </visual>
+        <visual>
+            <!-- STS3215 no-horn servo -->
+            <origin xyz="0 -0.042 0.031" rpy="${PI/2} 0 0"/>
+            <geometry><cylinder radius="0.018" length="0.040"/></geometry>
+            <material name="arm_servo"/>
+        </visual>
+        <collision>
+            <origin xyz="0 -0.028 0.018" rpy="0 0 0"/>
+            <geometry><box size="0.038 0.035 0.040"/></geometry>
+        </collision>
         <inertial>
             <origin xyz="-0.000103312 -0.0386143 0.0281156" rpy="0 0 0"/>
@@ -753,23 +731,6 @@
                      iyy="2.5391e-05" iyz="3.6412e-06" izz="2.1e-05"/>
         </inertial>
-        <visual>
-            <origin xyz="8.32667e-17 -0.0424 0.0306" rpy="1.5708 1.5708 0"/>
-            <geometry><mesh filename="package://omnibot_description/meshes/so101/sts3215_03a_no_horn_v1.stl"/></geometry>
-            <material name="arm_sts3215"/>
-        </visual>
-        <collision>
-            <origin xyz="8.32667e-17 -0.0424 0.0306" rpy="1.5708 1.5708 0"/>
-            <geometry><mesh filename="package://omnibot_description/meshes/so101/sts3215_03a_no_horn_v1.stl"/></geometry>
-        </collision>
-        <visual>
-            <origin xyz="0 -0.028 0.0181" rpy="-1.5708 -1.5708 0"/>
-            <geometry><mesh filename="package://omnibot_description/meshes/so101/wrist_roll_pitch_so101_v2.stl"/></geometry>
-            <material name="arm_3d_printed"/>
-        </visual>
-        <collision>
-            <origin xyz="0 -0.028 0.0181" rpy="-1.5708 -1.5708 0"/>
-            <geometry><mesh filename="package://omnibot_description/meshes/so101/wrist_roll_pitch_so101_v2.stl"/></geometry>
-        </collision>
-    </link>
+    </link>
+    <!-- wrist_flex — exact origin from so101_new_calib.urdf -->
     <joint name="arm_wrist_flex" type="revolute">
         <origin xyz="-0.1349 0.0052 3.62355e-17" rpy="4.02456e-15 8.67362e-16 -1.5708"/>
@@ -789,6 +750,22 @@
         </actuator>
     </transmission>
-    <!-- GRIPPER LINK (wrist_roll_follower + sts3215 roll servo) -->
+    <!-- GRIPPER — roll follower body + roll servo -->
     <link name="arm_gripper_link">
+        <visual>
+            <!-- Wrist roll follower body -->
+            <origin xyz="0 0 -0.015" rpy="0 0 0"/>
+            <geometry><box size="0.060 0.040 0.055"/></geometry>
+            <material name="arm_white"/>
+        </visual>
+        <visual>
+            <!-- STS3215 roll servo -->
+            <origin xyz="0.008 0 -0.023" rpy="0 ${PI/2} 0"/>
+            <geometry><cylinder radius="0.018" length="0.040"/></geometry>
+            <material name="arm_servo"/>
+        </visual>
+        <collision>
+            <origin xyz="0 0 -0.015" rpy="0 0 0"/>
+            <geometry><box size="0.060 0.040 0.055"/></geometry>
+        </collision>
         <inertial>
             <origin xyz="0.000213627 0.000245138 -0.025187" rpy="0 0 0"/>
@@ -797,23 +774,6 @@
                      iyy="4.33657e-05" iyz="-5.17847e-08" izz="3.45059e-05"/>
         </inertial>
-        <visual>
-            <origin xyz="0.0077 0.0001 -0.0234" rpy="-1.5708 -5.19179e-17 -1.66533e-16"/>
-            <geometry><mesh filename="package://omnibot_description/meshes/so101/sts3215_03a_v1.stl"/></geometry>
-            <material name="arm_sts3215"/>
-        </visual>
-        <collision>
-            <origin xyz="0.0077 0.0001 -0.0234" rpy="-1.5708 -5.19179e-17 -1.66533e-16"/>
-            <geometry><mesh filename="package://omnibot_description/meshes/so101/sts3215_03a_v1.stl"/></geometry>
-        </collision>
-        <visual>
-            <origin xyz="8.32667e-17 -0.000218214 0.000949706" rpy="-3.14159 -5.55112e-17 0"/>
-            <geometry><mesh filename="package://omnibot_description/meshes/so101/wrist_roll_follower_so101_v1.stl"/></geometry>
-            <material name="arm_3d_printed"/>
-        </visual>
-        <collision>
-            <origin xyz="8.32667e-17 -0.000218214 0.000949706" rpy="-3.14159 -5.55112e-17 0"/>
-            <geometry><mesh filename="package://omnibot_description/meshes/so101/wrist_roll_follower_so101_v1.stl"/></geometry>
-        </collision>
-    </link>
+    </link>
+    <!-- wrist_roll — exact origin from so101_new_calib.urdf -->
     <joint name="arm_wrist_roll" type="revolute">
         <origin xyz="5.55112e-17 -0.0611 0.0181" rpy="1.5708 0.0486795 3.14159"/>
@@ -833,10 +793,10 @@
         </actuator>
     </transmission>
-    <!-- GRIPPER FRAME (fixed dummy link — tool-frame reference) -->
+    <!-- GRIPPER FRAME — tool-frame reference (fixed, massless) -->
     <link name="arm_gripper_frame_link">
         <inertial>
             <origin xyz="0 0 0" rpy="0 0 0"/>
             <mass value="1e-9"/>
-            <inertia ixx="0" ixy="0" ixz="0" iyy="0" iyz="0" izz="0"/>
+            <inertia ixx="1e-9" ixy="0" ixz="0" iyy="1e-9" iyz="0" izz="1e-9"/>
         </inertial>
     </link>
@@ -845,8 +805,16 @@
         <parent link="arm_gripper_link"/>
         <child link="arm_gripper_frame_link"/>
-        <axis xyz="0 0 0"/>
-    </joint>
-    <!-- MOVING JAW LINK -->
+    </joint>
+    <!-- MOVING JAW -->
     <link name="arm_moving_jaw_link">
+        <visual>
+            <origin xyz="0 -0.030 0.019" rpy="0 0 0"/>
+            <geometry><box size="0.018 0.010 0.050"/></geometry>
+            <material name="arm_white"/>
+        </visual>
+        <collision>
+            <origin xyz="0 -0.030 0.019" rpy="0 0 0"/>
+            <geometry><box size="0.018 0.010 0.050"/></geometry>
+        </collision>
         <inertial>
             <origin xyz="-0.00157495 -0.0300244 0.0192755" rpy="0 0 0"/>
@@ -855,14 +823,6 @@
                      iyy="1.89032e-06" iyz="-1.09945e-07" izz="5.28738e-06"/>
         </inertial>
-        <visual>
-            <origin xyz="-5.55112e-17 -5.55112e-17 0.0189" rpy="9.53145e-17 6.93889e-18 1.24077e-24"/>
-            <geometry><mesh filename="package://omnibot_description/meshes/so101/moving_jaw_so101_v1.stl"/></geometry>
-            <material name="arm_3d_printed"/>
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
Commit message: fix(urdf): move OV9732 cameras to bottom plate, remove downward tilt
- Parent changed from top_plate_link → base_link (bottom plate)
- Pitch tilt removed (was -PI/6 downward, now 0 — faces straight out)

Co-Authored-By: Claude Sonnet 4.6 <noreply@anthropic.com>

File: robot_ws/src/omnibot_description/urdf/omnibot.urdf.xacro (robot description, xacro)
@@ -171,7 +171,6 @@
     <!-- ================================================================
          OV9732 wide-angle cameras — one on each side face of the chassis.
-         Mounted flush with the side faces of the top plate inside a
-         camera case. Each camera faces outward with a 30° downward tilt
-         for ground-obstacle coverage.
+         Mounted flush with the side faces of the bottom plate inside a
+         camera case. Each camera faces straight outward (no tilt).
          FOV: 100° (1.745 rad), 1280×720, USB UVC.
          ================================================================ -->
@@ -204,10 +203,10 @@
             </inertial>
         </link>
-        <!-- Parent: top_plate_link. Cameras sit on the side faces, at plate level. -->
+        <!-- Parent: base_link (bottom plate). Cameras sit on the side faces, facing straight out. -->
         <joint name="${prefix}_camera_joint" type="fixed">
-            <parent link="top_plate_link"/>
+            <parent link="base_link"/>
             <child link="${prefix}_camera_link"/>
             <origin xyz="${x_pos} ${y_pos} 0"
-                    rpy="0 ${-PI/6} ${yaw_angle}"/>
+                    rpy="0 0 ${yaw_angle}"/>
         </joint>
         <gazebo reference="${prefix}_camera_link">
