Commit message: update code

File: robot_ws/src/omnibot_description/urdf/omnibot.urdf.xacro (robot description, xacro)
@@ -34,4 +34,7 @@
         </inertial>
     </link>
+    <gazebo reference="base_link">
+        <material>Gazebo/Blue</material>
+    </gazebo>
     <joint name="base_footprint_joint" type="fixed">
         <parent link="base_footprint"/>
@@ -92,4 +95,9 @@
             </inertial>
         </link>
+        <gazebo reference="${prefix}_wheel_link">
+            <material>Gazebo/DarkGrey</material>
+            <mu1>0.8</mu1>
+            <mu2>0.8</mu2>
+        </gazebo>
         <joint name="${prefix}_wheel_joint" type="continuous">
             <parent link="base_link"/>
@@ -108,3 +116,31 @@
         </transmission>
     </xacro:macro>
-    <xacro:wheel prefix="front_left"  x_reflect="1"  y_reflect="1"  yaw_reflect="1"/>   <xacro:wheel prefix="front_right" x_reflect="1"  y_reflect="-1" yaw_reflect="-1"/>  <xacro:wheel prefix="rear_left"   x_reflect="-1" y_reflect="1"  yaw_reflect="-1"/>  <xacro:wheel prefix="rear_right"  x_reflect="-1" y_reflect="-1" yaw_reflect="1"/>   </robot>
+    <xacro:wheel prefix="front_left"  x_reflect="1"  y_reflect="1"  yaw_reflect="1"/>   <xacro:wheel prefix="front_right" x_reflect="1"  y_reflect="-1" yaw_reflect="-1"/>  <xacro:wheel prefix="rear_left"   x_reflect="-1" y_reflect="1"  yaw_reflect="-1"/>  <xacro:wheel prefix="rear_right"  x_reflect="-1" y_reflect="-1" yaw_reflect="1"/>
+    <!-- Gazebo Harmonic Mecanum Drive Plugin -->
+    <gazebo>
+        <plugin filename="gz-sim-mecanum-drive-system" name="gz::sim::systems::MecanumDrive">
+            <front_left_joint>front_left_wheel_joint</front_left_joint>
+            <front_right_joint>front_right_wheel_joint</front_right_joint>
+            <back_left_joint>rear_left_wheel_joint</back_left_joint>
+            <back_right_joint>rear_right_wheel_joint</back_right_joint>
+            <wheel_separation>${wheel_separation_y}</wheel_separation>
+            <wheelbase>${wheel_separation_x}</wheelbase>
+            <wheel_radius>${wheel_radius}</wheel_radius>
+            <odom_publish_frequency>50</odom_publish_frequency>
+            <!-- Leading slash = global topic scope, not model-namespaced -->
+            <topic>/cmd_vel</topic>
+            <odom_topic>/odom</odom_topic>
+            <tf_topic>/tf</tf_topic>
+            <frame_id>odom</frame_id>
+            <child_frame_id>base_footprint</child_frame_id>
+        </plugin>
+        <!-- Publish joint states -->
+        <plugin filename="gz-sim-joint-state-publisher-system" name="gz::sim::systems::JointStatePublisher">
+            <topic>joint_states</topic>
+            <joint_name>front_left_wheel_joint</joint_name>
+            <joint_name>front_right_wheel_joint</joint_name>
+            <joint_name>rear_left_wheel_joint</joint_name>
+            <joint_name>rear_right_wheel_joint</joint_name>
+        </plugin>
+    </gazebo>
+</robot>

Commit message: feat: add 5-camera multi-view setup with Bird's Eye View stitching
Integrates five OV9732 100° FOV USB cameras into OmniBot:
- 4 cameras on the mecanum base (front/rear/left/right)
- 1 wrist camera on the robotic arm

Key changes:
- bev_stitcher_node.py: new ROS 2 node that subscribes to 4 base camera
  topics and publishes a single /camera/base/bev/image_raw mosaic using
  OpenCV warpPerspective with alpha blending. Supports BEV homography
  calibration file (~/omnibot_bev_calibration.npz) with graceful fallback
  to a tiled quadrant layout when calibration is absent.
- mobile_manipulation.launch.py: replaces single front camera with 4 base
  cameras + wrist camera (all MJPEG to stay within RPi 5 USB bandwidth),
  and launches bev_stitcher_node automatically.
- smolvla_node.py: subscribe to BEV topic instead of /camera/front/;
  observation key renamed front -> bev throughout.
- teleop_recorder_node.py: record bev_image instead of front_image in
  both LeRobot HF dataset format and numpy fallback (.npz).
- omnibot.urdf.xacro: adds base_camera xacro macro (100° FOV, 30° ground
  tilt) instantiated for all four edges; adds wrist_camera_link; retains
  legacy camera_link for simulation.launch.py compatibility.
- setup.py: registers bev_stitcher_node console script entry point.

https://claude.ai/code/session_01Qzy7VsdkhW6uHZsxdY8ZNM

File: robot_ws/src/omnibot_description/urdf/omnibot.urdf.xacro (robot description, xacro)
@@ -9,5 +9,5 @@
     <xacro:property name="wheel_separation_x" value="0.165"/> <xacro:property name="wheel_separation_y" value="0.215"/> <xacro:property name="base_link_z_offset" value="${ground_clearance + chassis_height / 2.0}"/> <xacro:property name="wheel_z_offset" value="${wheel_radius - base_link_z_offset}"/> <xacro:property name="wheel_x_offset" value="${wheel_separation_x / 2.0}"/>
     <xacro:property name="wheel_y_offset" value="${wheel_separation_y / 2.0}"/>
-    <xacro:property name="camera_x_offset" value="0"/> <xacro:property name="camera_y_offset" value="0"/> <xacro:property name="camera_z_offset" value="${chassis_height / 2.0 + 0.01}"/> <xacro:property name="camera_size_x" value="0.06"/> <xacro:property name="camera_size_y" value="0.08"/> <xacro:property name="camera_size_z" value="0.04"/> <xacro:property name="base_mass" value="2.5"/> <xacro:property name="wheel_mass" value="0.2"/> <xacro:property name="camera_mass" value="0.3"/> <link name="base_footprint"/>
+    <xacro:property name="camera_x_offset" value="0"/> <xacro:property name="camera_y_offset" value="0"/> <xacro:property name="camera_z_offset" value="${chassis_height / 2.0 + 0.01}"/> <xacro:property name="camera_size_x" value="0.04"/> <xacro:property name="camera_size_y" value="0.025"/> <xacro:property name="camera_size_z" value="0.025"/> <xacro:property name="base_mass" value="2.5"/> <xacro:property name="wheel_mass" value="0.2"/> <xacro:property name="camera_mass" value="0.05"/> <link name="base_footprint"/>
     <link name="base_link">
         <visual>
@@ -42,6 +42,135 @@
         <origin xyz="0 0 ${base_link_z_offset}" rpy="0 0 0"/>
     </joint>
+    <!-- ================================================================
+         Base camera macro — instantiated 4× for front/rear/left/right.
+         OV9732: 100° FOV (1.745 rad), 1280×720, USB UVC.
+         Each camera sits on the top edge of the chassis, tilted ~30°
+         downward toward the ground plane for BEV capture.
+         ================================================================ -->
+    <xacro:macro name="base_camera" params="prefix x_pos y_pos yaw_angle">
+        <link name="${prefix}_camera_link">
+            <visual>
+                <origin xyz="0 0 0" rpy="0 0 0"/>
+                <geometry>
+                    <box size="${camera_size_x} ${camera_size_y} ${camera_size_z}"/>
+                </geometry>
+                <material name="dark_grey">
+                    <color rgba="0.2 0.2 0.2 1"/>
+                </material>
+            </visual>
+            <collision>
+                <origin xyz="0 0 0" rpy="0 0 0"/>
+                <geometry>
+                    <box size="${camera_size_x} ${camera_size_y} ${camera_size_z}"/>
+                </geometry>
+            </collision>
+            <inertial>
+                <mass value="${camera_mass}"/>
+                <origin xyz="0 0 0" rpy="0 0 0"/>
+                <inertia
+                    ixx="${camera_mass / 12.0 * (camera_size_y*camera_size_y + camera_size_z*camera_size_z)}"
+                    ixy="0.0" ixz="0.0"
+                    iyy="${camera_mass / 12.0 * (camera_size_x*camera_size_x + camera_size_z*camera_size_z)}"
+                    iyz="0.0"
+                    izz="${camera_mass / 12.0 * (camera_size_x*camera_size_x + camera_size_y*camera_size_y)}"/>
+            </inertial>
+        </link>
+        <!-- Tilt 30° downward (pitch = -PI/6) so cameras look at the ground -->
+        <joint name="${prefix}_camera_joint" type="fixed">
+            <parent link="base_link"/>
+            <child link="${prefix}_camera_link"/>
+            <origin xyz="${x_pos} ${y_pos} ${chassis_height / 2.0 + 0.015}"
+                    rpy="0 ${-PI/6} ${yaw_angle}"/>
+        </joint>
+        <!-- Gazebo camera sensor for simulation — 100° FOV, 1280×720 -->
+        <gazebo reference="${prefix}_camera_link">
+            <sensor name="${prefix}_camera_sensor" type="camera">
+                <always_on>1</always_on>
+                <update_rate>30</update_rate>
+                <visualize>false</visualize>
+                <topic>/camera/${prefix}/image_raw</topic>
+                <gz_frame_id>${prefix}_camera_link</gz_frame_id>
+                <camera>
+                    <horizontal_fov>1.745</horizontal_fov> <!-- 100 deg -->
+                    <image>
+                        <width>640</width>
+                        <height>480</height>
+                        <format>R8G8B8</format>
+                    </image>
+                    <clip>
+                        <near>0.05</near>
+                        <far>10</far>
+                    </clip>
+                </camera>
+            </sensor>
+        </gazebo>
+    </xacro:macro>
+    <!-- Instantiate 4 base cameras at the four edges of the chassis -->
+    <!-- Front: centre of forward edge, facing forward (yaw=0) -->
+    <xacro:base_camera prefix="front"
+        x_pos="${chassis_length / 2.0 - 0.01}"
+        y_pos="0"
+        yaw_angle="0"/>
+    <!-- Rear: centre of rear edge, facing backward (yaw=PI) -->
+    <xacro:base_camera prefix="rear"
+        x_pos="${-(chassis_length / 2.0 - 0.01)}"
+        y_pos="0"
+        yaw_angle="${PI}"/>
+    <!-- Left: centre of left edge, facing left (yaw=PI/2) -->
+    <xacro:base_camera prefix="left"
+        x_pos="0"
+        y_pos="${chassis_width / 2.0 - 0.01}"
+        yaw_angle="${PI/2}"/>
+    <!-- Right: centre of right edge, facing right (yaw=-PI/2) -->
+    <xacro:base_camera prefix="right"
+        x_pos="0"
+        y_pos="${-(chassis_width / 2.0 - 0.01)}"
+        yaw_angle="${-PI/2}"/>
+    <!-- ================================================================
+         Wrist camera link — mounted on the arm end-effector.
+         Defined as a separate fixed link relative to wrist_link.
+         The arm URDF (omnibot_arm package) provides wrist_link; this
+         joint connects to it when the arm is loaded in the same URDF.
+         For standalone robot description without arm, this link is
+         kept as a child of base_link as a placeholder.
+         ================================================================ -->
+    <link name="wrist_camera_link">
+        <visual>
+            <origin xyz="0 0 0" rpy="0 0 0"/>
+            <geometry>
+                <box size="${camera_size_x} ${camera_size_y} ${camera_size_z}"/>
+            </geometry>
+            <material name="dark_grey_wrist">
+                <color rgba="0.2 0.2 0.2 1"/>
+            </material>
+        </visual>
+        <collision>
+            <origin xyz="0 0 0" rpy="0 0 0"/>
+            <geometry>
+                <box size="${camera_size_x} ${camera_size_y} ${camera_size_z}"/>
+            </geometry>
+        </collision>
+        <inertial>
+            <mass value="${camera_mass}"/>
+            <origin xyz="0 0 0" rpy="0 0 0"/>
+            <inertia
+                ixx="${camera_mass / 12.0 * (camera_size_y*camera_size_y + camera_size_z*camera_size_z)}"
+                ixy="0.0" ixz="0.0"
+                iyy="${camera_mass / 12.0 * (camera_size_x*camera_size_x + camera_size_z*camera_size_z)}"
+                iyz="0.0"
+                izz="${camera_mass / 12.0 * (camera_size_x*camera_size_x + camera_size_y*camera_size_y)}"/>
+        </inertial>
+    </link>
+    <!-- Placeholder joint: wrist camera on base_link until arm URDF is merged -->
+    <joint name="wrist_camera_joint" type="fixed">
+        <parent link="base_link"/>
+        <child link="wrist_camera_link"/>
+        <origin xyz="${chassis_length / 2.0 + 0.02} 0 ${chassis_height / 2.0 + 0.08}"
+                rpy="0 ${PI/4} 0"/>
+    </joint>
+    <!-- Gazebo simulation sensor — mounted on camera_link, publishes /camera/image_raw -->
+    <!-- Kept for backwards-compatibility with simulation.launch.py -->
     <link name="camera_link">
-         <visual>
+        <visual>
             <origin xyz="0 0 0" rpy="0 0 0"/>
             <geometry>
@@ -53,15 +182,18 @@
         </visual>
         <collision>
-             <origin xyz="0 0 0" rpy="0 0 0"/>
-             <geometry>
+            <origin xyz="0 0 0" rpy="0 0 0"/>
+            <geometry>
                 <box size="${camera_size_x} ${camera_size_y} ${camera_size_z}"/>
             </geometry>
         </collision>
-         <inertial>
+        <inertial>
             <mass value="${camera_mass}"/>
             <origin xyz="0 0 0" rpy="0 0 0"/>
-            <inertia ixx="${camera_mass / 12.0 * (camera_size_y*camera_size_y + camera_size_z*camera_size_z)}" ixy="0.0" ixz="0.0"
-                     iyy="${camera_mass / 12.0 * (camera_size_x*camera_size_x + camera_size_z*camera_size_z)}" iyz="0.0"
-                     izz="${camera_mass / 12.0 * (camera_size_x*camera_size_x + camera_size_y*camera_size_y)}" />
+            <inertia
+                ixx="${camera_mass / 12.0 * (camera_size_y*camera_size_y + camera_size_z*camera_size_z)}"
+                ixy="0.0" ixz="0.0"
+                iyy="${camera_mass / 12.0 * (camera_size_x*camera_size_x + camera_size_z*camera_size_z)}"
+                iyz="0.0"
+                izz="${camera_mass / 12.0 * (camera_size_x*camera_size_x + camera_size_y*camera_size_y)}"/>
         </inertial>
     </link>
@@ -69,5 +201,6 @@
         <parent link="base_link"/>
         <child link="camera_link"/>
-        <origin xyz="${camera_x_offset} ${camera_y_offset} ${camera_z_offset}" rpy="0 0 0"/> </joint>
+        <origin xyz="${camera_x_offset} ${camera_y_offset} ${camera_z_offset}" rpy="0 0 0"/>
+    </joint>
     <!-- Gazebo Camera Sensor — mounted on camera_link, publishes /camera/image_raw -->
     <gazebo reference="camera_link">

Commit message: Add 3-D mapping stack: RTAB-Map + OctoMap + RealSense D435 depth camera
- omnibot.urdf.xacro: add Intel RealSense D435 depth camera link, optical
  frame, and Gazebo Harmonic rgbd_camera sensor (69° FOV, 0.1–10 m range)
  mounted at the front of the chassis

- rtabmap_params.yaml: RGB-D SLAM config — 5 cm grid cells, OctoMap output,
  loop-closure via bag-of-words, approx_sync for RGB-D pair matching

- octomap_params.yaml: octomap_server config — consumes /rtabmap/cloud_map,
  5 cm resolution, ground filtering, publishes /projected_map (2-D slice)

- rtabmap.launch.py: launches rtabmap core + octomap_server +
  depth_image_proc point cloud node; conditional on use_3d_mapping arg

- nav2_params.yaml: add PointCloud2 observation source (/camera/depth/points)
  to VoxelLayer (local costmap) and ObstacleLayer (global costmap) alongside
  the existing LaserScan source for richer 3-D obstacle awareness

- ros_gz_bridge.yaml: bridge Gazebo RGBD sensor topics to ROS 2
  (/camera/depth/image, /camera/depth/camera_info, /camera/depth/points)

- autonomous_robot.launch.py: add use_3d_mapping:=false arg; set true to
  co-launch RTAB-Map alongside slam_toolbox

- package.xml: add rtabmap_ros, octomap_server, pcl_ros, depth_image_proc,
  octomap_msgs dependencies

Usage:
  ros2 launch omnibot_navigation autonomous_robot.launch.py use_3d_mapping:=true

https://claude.ai/code/session_01Qzy7VsdkhW6uHZsxdY8ZNM

File: robot_ws/src/omnibot_description/urdf/omnibot.urdf.xacro (robot description, xacro)
@@ -222,4 +222,82 @@
                     <far>50</far>
                 </clip>
+            </camera>
+        </sensor>
+    </gazebo>
+    <!-- ================================================================
+         Intel RealSense D435 Depth Camera
+         Mounted at the front-centre of the chassis, facing forward.
+         Used for 3-D mapping (RTAB-Map) and obstacle avoidance.
+         D435 specs: depth FOV 69°H × 42°V, range 0.1 – 10 m
+         RGB FOV: ~69°H × 42°V
+         ================================================================ -->
+    <xacro:property name="depth_cam_x"  value="${chassis_length / 2.0 - 0.005}"/>
+    <xacro:property name="depth_cam_z"  value="${chassis_height / 2.0 + 0.015}"/>
+    <xacro:property name="depth_cam_mass" value="0.072"/>
+    <!-- Optical frame (Z forward, X right, Y down) -->
+    <link name="depth_camera_link">
+        <visual>
+            <origin xyz="0 0 0" rpy="0 0 0"/>
+            <geometry>
+                <box size="0.090 0.025 0.025"/>
+            </geometry>
+            <material name="realsense_grey">
+                <color rgba="0.15 0.15 0.15 1"/>
+            </material>
+        </visual>
+        <collision>
+            <origin xyz="0 0 0" rpy="0 0 0"/>
+            <geometry>
+                <box size="0.090 0.025 0.025"/>
+            </geometry>
+        </collision>
+        <inertial>
+            <mass value="${depth_cam_mass}"/>
+            <origin xyz="0 0 0" rpy="0 0 0"/>
+            <inertia
+                ixx="${depth_cam_mass / 12.0 * (0.025*0.025 + 0.025*0.025)}"
+                ixy="0" ixz="0"
+                iyy="${depth_cam_mass / 12.0 * (0.090*0.090 + 0.025*0.025)}"
+                iyz="0"
+                izz="${depth_cam_mass / 12.0 * (0.090*0.090 + 0.025*0.025)}"/>
+        </inertial>
+    </link>
+    <joint name="depth_camera_joint" type="fixed">
+        <parent link="base_link"/>
+        <child link="depth_camera_link"/>
+        <origin xyz="${depth_cam_x} 0 ${depth_cam_z}" rpy="0 0 0"/>
+    </joint>
+    <!-- Optical frame: rotate 90° so Z points forward in ROS convention -->
+    <link name="depth_camera_optical_frame"/>
+    <joint name="depth_camera_optical_joint" type="fixed">
+        <parent link="depth_camera_link"/>
+        <child link="depth_camera_optical_frame"/>
+        <origin xyz="0 0 0" rpy="${-PI/2} 0 ${-PI/2}"/>
+    </joint>
+    <!-- Gazebo Harmonic RGBD sensor (models D435 RGB-D) -->
+    <gazebo reference="depth_camera_link">
+        <sensor name="depth_camera_sensor" type="rgbd_camera">
+            <always_on>1</always_on>
+            <update_rate>15</update_rate>
+            <visualize>false</visualize>
+            <topic>/camera/depth</topic>
+            <gz_frame_id>depth_camera_link</gz_frame_id>
+            <camera>
+                <!-- D435 depth horizontal FOV ~69° = 1.2043 rad -->
+                <horizontal_fov>1.2043</horizontal_fov>
+                <image>
+                    <width>640</width>
+                    <height>480</height>
+                    <format>R_FLOAT32</format>
+                </image>
+                <clip>
+                    <near>0.1</near>
+                    <far>10.0</far>
+                </clip>
+                <noise>
+                    <type>gaussian</type>
+                    <mean>0.0</mean>
+                    <stddev>0.01</stddev>
+                </noise>
             </camera>
         </sensor>
