Commit message: Switch 3-D mapping depth camera from RealSense D435 to Orbbec Astra Pro
URDF (omnibot.urdf.xacro):
- Replace D435 link with Astra Pro body (165×30×40 mm, 300 g)
- Update FOV: 69° → 60° (1.0472 rad horizontal)
- Update depth range: 0.1–10 m → 0.6–8.0 m
- Add 12° downward tilt so camera captures obstacles at mid-range
- Rename Gazebo sensor to astra_pro_sensor

rtabmap_params.yaml:
- Update Grid/RangeMin: 0.1 → 0.6  (Astra blind zone)
- Update Grid/RangeMax: 5.0 → 8.0  (Astra max range)
- Update header comments to document Astra Pro topic layout

rtabmap.launch.py:
- Add astra_camera_node (ros2_astra_camera driver, skipped in sim)
- Fix RTAB-Map remappings: rgb/image → /camera/color/image_raw,
  depth/image → /camera/depth/image_raw (proper RGB-D pair)
- Remove depth_image_proc node (Astra driver publishes points natively)
- Add build-from-source install instructions in module docstring

ros_gz_bridge.yaml:
- Rename depth image bridge: /camera/depth/image → /camera/depth/image_raw
- Add /camera/color/image_raw bridge (from Gazebo image_rgb8 output)
- Add /camera/color/camera_info bridge
- Update comments to reference Astra Pro

octomap_params.yaml:
- Update sensor_model_max_range: 5.0 → 8.0

nav2_params.yaml:
- Update pointcloud raytrace/obstacle ranges to match Astra 0.6–8.0 m

package.xml:
- Replace depth_image_proc with astra_camera exec_depend + build instructions

https://claude.ai/code/session_01Qzy7VsdkhW6uHZsxdY8ZNM

File: robot_ws/src/omnibot_description/urdf/omnibot.urdf.xacro (robot description, xacro)
@@ -226,22 +226,26 @@
     </gazebo>
     <!-- ================================================================
-         Intel RealSense D435 Depth Camera
-         Mounted at the front-centre of the chassis, facing forward.
-         Used for 3-D mapping (RTAB-Map) and obstacle avoidance.
-         D435 specs: depth FOV 69°H × 42°V, range 0.1 – 10 m
-         RGB FOV: ~69°H × 42°V
+         Orbbec Astra Pro Depth Camera
+         Mounted at the front-centre of the chassis, facing forward,
+         tilted 12° downward to ensure ground obstacles within 0.6 m
+         blind zone are captured on the sides by the OV9732 cameras.
+         Astra Pro specs:
+           Depth: 640×480 @ 30 fps, FOV 60°H × 49.5°V, range 0.6–8.0 m
+           RGB  : 1280×960 @ 30 fps, FOV 60°H × 49.5°V
+           Body : 165 mm × 30 mm × 40 mm, 300 g, USB 2.0
+         ROS 2 driver: https://github.com/orbbec/ros2_astra_camera
          ================================================================ -->
-    <xacro:property name="depth_cam_x"  value="${chassis_length / 2.0 - 0.005}"/>
-    <xacro:property name="depth_cam_z"  value="${chassis_height / 2.0 + 0.015}"/>
-    <xacro:property name="depth_cam_mass" value="0.072"/>
-    <!-- Optical frame (Z forward, X right, Y down) -->
+    <xacro:property name="astra_x"    value="${chassis_length / 2.0 - 0.005}"/>
+    <xacro:property name="astra_z"    value="${chassis_height / 2.0 + 0.020}"/>
+    <xacro:property name="astra_mass" value="0.300"/>
     <link name="depth_camera_link">
         <visual>
             <origin xyz="0 0 0" rpy="0 0 0"/>
             <geometry>
-                <box size="0.090 0.025 0.025"/>
-            </geometry>
-            <material name="realsense_grey">
-                <color rgba="0.15 0.15 0.15 1"/>
+                <!-- Astra Pro body: 165 mm wide × 30 mm deep × 40 mm tall -->
+                <box size="0.030 0.165 0.040"/>
+            </geometry>
+            <material name="astra_black">
+                <color rgba="0.08 0.08 0.08 1"/>
             </material>
         </visual>
@@ -249,24 +253,26 @@
             <origin xyz="0 0 0" rpy="0 0 0"/>
             <geometry>
-                <box size="0.090 0.025 0.025"/>
+                <box size="0.030 0.165 0.040"/>
             </geometry>
         </collision>
         <inertial>
-            <mass value="${depth_cam_mass}"/>
+            <mass value="${astra_mass}"/>
             <origin xyz="0 0 0" rpy="0 0 0"/>
             <inertia
-                ixx="${depth_cam_mass / 12.0 * (0.025*0.025 + 0.025*0.025)}"
+                ixx="${astra_mass / 12.0 * (0.165*0.165 + 0.040*0.040)}"
                 ixy="0" ixz="0"
-                iyy="${depth_cam_mass / 12.0 * (0.090*0.090 + 0.025*0.025)}"
+                iyy="${astra_mass / 12.0 * (0.030*0.030 + 0.040*0.040)}"
                 iyz="0"
-                izz="${depth_cam_mass / 12.0 * (0.090*0.090 + 0.025*0.025)}"/>
+                izz="${astra_mass / 12.0 * (0.030*0.030 + 0.165*0.165)}"/>
         </inertial>
     </link>
+    <!-- Tilt 12° downward (pitch = -0.2094 rad) so the camera sees ground
+         obstacles starting at ~2.8 m while still covering the full scene -->
     <joint name="depth_camera_joint" type="fixed">
         <parent link="base_link"/>
         <child link="depth_camera_link"/>
-        <origin xyz="${depth_cam_x} 0 ${depth_cam_z}" rpy="0 0 0"/>
-    </joint>
-    <!-- Optical frame: rotate 90° so Z points forward in ROS convention -->
+        <origin xyz="${astra_x} 0 ${astra_z}" rpy="0 -0.2094 0"/>
+    </joint>
+    <!-- Optical frame: Z forward, X right, Y down (ROS convention) -->
     <link name="depth_camera_optical_frame"/>
     <joint name="depth_camera_optical_joint" type="fixed">
@@ -275,15 +281,23 @@
         <origin xyz="0 0 0" rpy="${-PI/2} 0 ${-PI/2}"/>
     </joint>
-    <!-- Gazebo Harmonic RGBD sensor (models D435 RGB-D) -->
+    <!-- Gazebo Harmonic RGBD sensor (models Astra Pro RGB-D)
+         Publishes:
+           /camera/depth/image      — 16-bit depth (mm)  → bridged as image_raw
+           /camera/depth/points     — PointCloud2
+           /camera/color/image_raw  — RGB 640×480
+         These topic names are chosen to match the real ros2_astra_camera driver
+         output so that rtabmap.launch.py remappings work identically in
+         simulation and on the physical robot. -->
     <gazebo reference="depth_camera_link">
-        <sensor name="depth_camera_sensor" type="rgbd_camera">
+        <sensor name="astra_pro_sensor" type="rgbd_camera">
             <always_on>1</always_on>
-            <update_rate>15</update_rate>
+            <update_rate>30</update_rate>
             <visualize>false</visualize>
+            <!-- Base topic; Gazebo appends /image, /points, /camera_info -->
             <topic>/camera/depth</topic>
-            <gz_frame_id>depth_camera_link</gz_frame_id>
+            <gz_frame_id>depth_camera_optical_frame</gz_frame_id>
             <camera>
-                <!-- D435 depth horizontal FOV ~69° = 1.2043 rad -->
-                <horizontal_fov>1.2043</horizontal_fov>
+                <!-- Astra Pro horizontal FOV 60° = 1.0472 rad -->
+                <horizontal_fov>1.0472</horizontal_fov>
                 <image>
                     <width>640</width>
@@ -292,11 +306,12 @@
                 </image>
                 <clip>
-                    <near>0.1</near>
-                    <far>10.0</far>
+                    <!-- Astra Pro minimum range 0.6 m -->
+                    <near>0.6</near>
+                    <far>8.0</far>
                 </clip>
                 <noise>
                     <type>gaussian</type>
                     <mean>0.0</mean>
-                    <stddev>0.01</stddev>
+                    <stddev>0.005</stddev>
                 </noise>
             </camera>

Commit message: Add digital twin infrastructure for contributor onboarding
- Add 2D lidar (RPLidar A1 sim) to URDF xacro + omnibot_world.sdf plugin
- Bridge /scan (LaserScan) via ros_gz_bridge.yaml — unblocks SLAM/Nav2 contributors
- Update simulation.launch.py: BEV stitcher, ROSBridge, Foxglove bridge,
  world/rviz/rosbridge/foxglove/bev launch args, IfCondition guards
- Add digital_twin/ directory:
    worlds/omnibot_lab.sdf     : 2-room indoor lab with table + 4 YCB objects
    configs/nav2_sim_params.yaml : sim-tuned Nav2 (use_sim_time, tighter inflation)
    configs/rviz/perception.rviz : camera feeds, depth, BEV, pointcloud
    configs/rviz/navigation.rviz : map, costmap, path, lidar, nav2 panel
    configs/rviz/manipulation.rviz : arm TF, joint states, wrist camera
    configs/foxglove/omnibot_layout.json : browser visualization layout
    docker/Dockerfile.sim       : Ubuntu 24.04 + ROS Jazzy + Gazebo Harmonic
    docker/docker-compose.yml   : headless sim + foxglove services
    docker/docker-compose.gpu.yml : NVIDIA GPU override
    docker/post_create.sh       : rosdep + colcon bootstrap script
    scripts/build_usd.sh        : automates xacro→URDF bake + Isaac Sim steps
    scripts/setup_omnigraph.py  : wires OmniGraph ROS 2 action graph in Isaac Sim
    scenarios/pick_and_place.yaml : 5 VLA/manipulation scenarios
    scenarios/nav_corridor.yaml   : 5 navigation benchmark scenarios
    README.md                   : contributor quick-start guide
- Add .devcontainer/devcontainer.json for VS Code Dev Containers

https://claude.ai/code/session_01JowjBXS9GZcuD8S9f6T4PZ

File: robot_ws/src/omnibot_description/urdf/omnibot.urdf.xacro (robot description, xacro)
@@ -920,3 +920,71 @@
              plugins loaded in omnibot_world.sdf — do NOT duplicate here. -->
     </gazebo>
+    <!-- ================================================================
+         2D Lidar — RPLidar A1 (simulated)
+         Mounted on top plate, front-centre, clear of the arm base.
+         Provides /scan (sensor_msgs/LaserScan) for SLAM Toolbox and Nav2.
+         Physical: 360° @ 5.5 Hz, 12 m range.
+         Sim model: 360 rays, 10 Hz, 12 m max range, small Gaussian noise.
+         gz-sim-sensors-system is already loaded at world level in
+         omnibot_world.sdf — no duplicate plugin needed here.
+         ================================================================ -->
+    <link name="lidar_link">
+        <visual>
+            <origin xyz="0 0 0" rpy="0 0 0"/>
+            <geometry>
+                <cylinder radius="0.038" length="0.035"/>
+            </geometry>
+            <material name="lidar_black">
+                <color rgba="0.08 0.08 0.08 1"/>
+            </material>
+        </visual>
+        <collision>
+            <origin xyz="0 0 0" rpy="0 0 0"/>
+            <geometry>
+                <cylinder radius="0.038" length="0.035"/>
+            </geometry>
+        </collision>
+        <inertial>
+            <mass value="0.17"/>
+            <origin xyz="0 0 0" rpy="0 0 0"/>
+            <inertia ixx="1e-4" ixy="0" ixz="0" iyy="1e-4" iyz="0" izz="1e-4"/>
+        </inertial>
+    </link>
+    <!-- Mounted on rear half of top plate (x < 0) so the arm does not
+         occlude the beam.  Z puts the scan plane ~18 mm above top surface. -->
+    <joint name="lidar_joint" type="fixed">
+        <parent link="top_plate_link"/>
+        <child link="lidar_link"/>
+        <origin xyz="${-(chassis_length / 2.0 - 0.06)} 0 ${plate_thickness / 2.0 + 0.018}"
+                rpy="0 0 0"/>
+    </joint>
+    <gazebo reference="lidar_link">
+        <sensor name="lidar_sensor" type="gpu_lidar">
+            <always_on>1</always_on>
+            <update_rate>10</update_rate>
+            <visualize>false</visualize>
+            <topic>/scan</topic>
+            <gz_frame_id>lidar_link</gz_frame_id>
+            <lidar>
+                <scan>
+                    <horizontal>
+                        <samples>360</samples>
+                        <resolution>1</resolution>
+                        <min_angle>-3.14159</min_angle>
+                        <max_angle>3.14159</max_angle>
+                    </horizontal>
+                </scan>
+                <range>
+                    <min>0.15</min>
+                    <max>12.0</max>
+                    <resolution>0.01</resolution>
+                </range>
+                <noise>
+                    <type>gaussian</type>
+                    <mean>0.0</mean>
+                    <stddev>0.01</stddev>
+                </noise>
+            </lidar>
+        </sensor>
+    </gazebo>
 </robot>

Commit message: Fix: remove fake 2D lidar, use depthimage_to_laserscan instead
OmniBot has no physical lidar. The previous commit incorrectly added a
simulated RPLidar A1 link to the URDF — reverted completely.

/scan (LaserScan) for slam_toolbox and Nav2 is now generated by
depthimage_to_laserscan_node, converting the Orbbec Astra Pro depth
image (/camera/depth/image_raw → /scan). This matches real hardware
behaviour and keeps simulation and physical robot on identical pipelines.

Changes:
- Remove lidar_link / lidar_joint / gpu_lidar sensor from URDF xacro
- Remove gz-sim-gpu-lidar-system plugin from omnibot_world.sdf
- Replace /scan bridge entry in ros_gz_bridge.yaml with explanatory comment
- Add depthimage_to_laserscan_node to simulation.launch.py (step 6)
- Update nav2_sim_params.yaml comment to reflect correct /scan source

https://claude.ai/code/session_01JowjBXS9GZcuD8S9f6T4PZ

File: robot_ws/src/omnibot_description/urdf/omnibot.urdf.xacro (robot description, xacro)
@@ -920,71 +920,3 @@
              plugins loaded in omnibot_world.sdf — do NOT duplicate here. -->
     </gazebo>
-    <!-- ================================================================
-         2D Lidar — RPLidar A1 (simulated)
-         Mounted on top plate, front-centre, clear of the arm base.
-         Provides /scan (sensor_msgs/LaserScan) for SLAM Toolbox and Nav2.
-         Physical: 360° @ 5.5 Hz, 12 m range.
-         Sim model: 360 rays, 10 Hz, 12 m max range, small Gaussian noise.
-         gz-sim-sensors-system is already loaded at world level in
-         omnibot_world.sdf — no duplicate plugin needed here.
-         ================================================================ -->
-    <link name="lidar_link">
-        <visual>
-            <origin xyz="0 0 0" rpy="0 0 0"/>
-            <geometry>
-                <cylinder radius="0.038" length="0.035"/>
-            </geometry>
-            <material name="lidar_black">
-                <color rgba="0.08 0.08 0.08 1"/>
-            </material>
-        </visual>
-        <collision>
-            <origin xyz="0 0 0" rpy="0 0 0"/>
-            <geometry>
-                <cylinder radius="0.038" length="0.035"/>
-            </geometry>
-        </collision>
-        <inertial>
-            <mass value="0.17"/>
-            <origin xyz="0 0 0" rpy="0 0 0"/>
-            <inertia ixx="1e-4" ixy="0" ixz="0" iyy="1e-4" iyz="0" izz="1e-4"/>
-        </inertial>
-    </link>
-    <!-- Mounted on rear half of top plate (x < 0) so the arm does not
-         occlude the beam.  Z puts the scan plane ~18 mm above top surface. -->
-    <joint name="lidar_joint" type="fixed">
-        <parent link="top_plate_link"/>
-        <child link="lidar_link"/>
-        <origin xyz="${-(chassis_length / 2.0 - 0.06)} 0 ${plate_thickness / 2.0 + 0.018}"
-                rpy="0 0 0"/>
-    </joint>
-    <gazebo reference="lidar_link">
-        <sensor name="lidar_sensor" type="gpu_lidar">
-            <always_on>1</always_on>
-            <update_rate>10</update_rate>
-            <visualize>false</visualize>
-            <topic>/scan</topic>
-            <gz_frame_id>lidar_link</gz_frame_id>
-            <lidar>
-                <scan>
-                    <horizontal>
-                        <samples>360</samples>
-                        <resolution>1</resolution>
-                        <min_angle>-3.14159</min_angle>
-                        <max_angle>3.14159</max_angle>
-                    </horizontal>
-                </scan>
-                <range>
-                    <min>0.15</min>
-                    <max>12.0</max>
-                    <resolution>0.01</resolution>
-                </range>
-                <noise>
-                    <type>gaussian</type>
-                    <mean>0.0</mean>
-                    <stddev>0.01</stddev>
-                </noise>
-            </lidar>
-        </sensor>
-    </gazebo>
 </robot>
